File: hardware/motor-driver/pcb/motor-driver.kicad_pcb (KiCad board)
At the start: 2 copper layers, 9 parts, among them M2_1 M2, M2_2 M2, U1 XT30PW-F, U2 X1311WV-10J-C40D24, U3 X1311WV-10J-C40D24

Commit message: bottom plate schematic, and removed some random stuff
Other:
- board outline added: 19.1 x 17.6 mm
