File: hardware/kicker/bottom-pcb/pcb.kicad_sch (KiCad schematic)
At the start: 23 parts, among them J1 Conn_01x05, Q1 NMOS, U2 TS4535TP 250GF 009, U4 TC4427AEOA713_C5804606

Commit message: quite a few changes
Parts:
- removed 48VPWR1, VCCPWR1: Conn_01x04, Connector_PinHeader_2.54mm:PinHeader_1x04_P2.54mm_Vertical, symbol Connector_Generic:Conn_01x04
- removed J1: Conn_01x05, Connector_PinHeader_2.54mm:PinHeader_1x05_P2.54mm_Vertical, symbol Connector_Generic:Conn_01x05
- added C2, C3: 1uF, Capacitor_SMD:C_1206_3216Metric_Pad1.33x1.80mm_HandSolder, symbol Device:C
- added D1: MBRD1045, EasyEDA:TO-252-3_L6.5-W5.9-P4.60-LS10.0-BL, symbol EasyEDA:MBRD1045
- added H3, H4: MountingHole_Pad, MountingHole:MountingHole_2.2mm_M2_Pad_Via, symbol Mechanical:MountingHole_Pad
- added J1, J2: Conn_01x04, Connector_PinSocket_2.54mm:PinSocket_1x04_P2.54mm_Vertical, symbol Connector_Generic:Conn_01x04
- added J3: Conn_01x02, Connector_JST:JST_PH_B2B-PH-K_1x02_P2.00mm_Vertical, symbol Connector_Generic:Conn_01x02
- added L1: SMDRI127-470MT, EasyEDA:IND-SMD_L12.3-W12.3, symbol EasyEDA:SMDRI127-470MT
- added R5: 10k, Resistor_SMD:R_1206_3216Metric_Pad1.30x1.75mm_HandSolder, symbol Device:R
- added R6: 73.2kR, Resistor_SMD:R_1206_3216Metric_Pad1.30x1.75mm_HandSolder, symbol Device:R
- added R7: 2kR, Resistor_SMD:R_1206_3216Metric_Pad1.30x1.75mm_HandSolder, symbol Device:R
- added R8: 10kR, Resistor_SMD:R_1206_3216Metric_Pad1.30x1.75mm_HandSolder, symbol Device:R
- added U1: XL6019E1, EasyEDA:TO-263-5_L10.2-W9.9-P1.70-LS14.4-TL, symbol EasyEDA:XL6019E1
Connections:
- net +48V: now also R10.1, R9.2, C3.1, D1.2 (K), R6.1, R8.1; no longer R10.2, R9.1
- net CAP_VCC: now also R10.2, R9.1; no longer R10.1, R9.2
- net GND: now also C2.1, C3.2, J1.3 (Pin_3), J1.4 (Pin_4), J2.4 (Pin_4), J3.2 (Pin_2), R7.2, R8.2, U1.1 (GND)
- net INA: now also J2.3 (Pin_3)
- net INB: now also J2.2 (Pin_2)
- net OUTA: no longer D2.2 (A)
- net OUTB: now also J3.1 (Pin_1)
- net VCC: now also C2.2, J1.1 (Pin_1), J1.2 (Pin_2), J2.1 (Pin_1), L1.2, R5.2, U1.4 (VIN)
- net at KICK1.2 (Pin_2), Q1.1 (D): now also D2.2 (A)
- new net: R5.1, U1.2 (EN)
- new net: D1.1 (A), D1.3 (A), L1.1, U1.3 (SW), U1.6 (SW)
- new net FB: R6.2, R7.1, U1.5 (FB)
- no-connect marks 4 -> 6
Other:
- moved on the sheet: C1, D2, R10, R9
