File: hardware/bottom-plate/pcb/pcb.kicad_pcb (KiCad board)
At the start: 2 copper layers, 64 x 63.5 mm, 117 parts, among them U1 Pico, U2 CD4051B

Commit message: kicker pcb done, working on bottom plate
Parts:
- removed DRV0: ~, custom:DRV8224_breakout
- removed KICK_PWR1: XT30-F, Connector_AMASS:AMASS_XT30U-F_1x02_P5.0mm_Vertical
- removed MUX1, MUX2, MUX3: CD74HC4067M, Package_SO:SOIC-24W_7.5x15.4mm_P1.27mm
- removed PWR0: XT60-M, Connector_AMASS:AMASS_XT60-M_1x02_P7.20mm_Vertical
- removed REF**: PMW3360_breakout, custom:PMW3360_breakout
- removed U2: CD4051B, Package_SO:SOIC-16_3.9x9.9mm_P1.27mm
- added AMUX1: CD74HC4067M, Package_SO:SOIC-24W_7.5x15.4mm_P1.27mm, F.Cu at (191.9, -2.96)
- added AMUX2: CD74HC4067M, Package_SO:SOIC-24W_7.5x15.4mm_P1.27mm, F.Cu at (204.8, -2.96)
- added AMUX3: CD74HC4067M, Package_SO:SOIC-24W_7.5x15.4mm_P1.27mm, F.Cu at (217.7, -2.96)
- added BUCK1: ~, custom:mini560, F.Cu at (0.00, 45.0)
- added C1: 150uF, Capacitor_SMD:CP_Elec_6.3x7.7, F.Cu at (213.0, 63.2)
- added C2: 22uF, PCM_Capacitor_SMD_AKL:C_0805_2012Metric_Pad1.15x1.40mm_HandSolder, F.Cu at (205.4, 52.3)
- added C3: 1uF, PCM_Capacitor_SMD_AKL:C_0805_2012Metric_Pad1.15x1.40mm_HandSolder, F.Cu at (205.4, 55.4)
- added C4: 10uF, PCM_Capacitor_SMD_AKL:C_0805_2012Metric_Pad1.15x1.40mm_HandSolder, F.Cu at (205.4, 58.4)
- added CTRL1: Conn_01x04, Connector_JST:JST_XH_B4B-XH-A_1x04_P2.50mm_Vertical, F.Cu at (161.7, 3.41)
- added DMUX1: MCP23S17_SO, Package_SO:SOIC-28W_7.5x17.9mm_P1.27mm, F.Cu at (150.3, -9.69)
- added DMUX2: MCP23S17_SO, Package_SO:SOIC-28W_7.5x17.9mm_P1.27mm, F.Cu at (163.2, -9.69)
- added KICK1: ~, custom:kicker, F.Cu at (0.00, 10.3)
- added LDO1: TLV1117-33, Package_TO_SOT_SMD:SOT-223-3_TabPin2, F.Cu at (212.7, 55.0)
- added LED1: 10mA 2.7-3.5V, Diode_SMD:D_0603_1608Metric_Pad1.05x0.95mm_HandSolder, F.Cu at (187.7, -38.1)
- added LED10: 10mA 2.7-3.5V, Diode_SMD:D_0603_1608Metric_Pad1.05x0.95mm_HandSolder, F.Cu at (187.7, -14.8)
- added LED11: 10mA 2.7-3.5V, Diode_SMD:D_0603_1608Metric_Pad1.05x0.95mm_HandSolder, F.Cu at (192.1, -38.1)
- added LED12: 10mA 2.7-3.5V, Diode_SMD:D_0603_1608Metric_Pad1.05x0.95mm_HandSolder, F.Cu at (192.1, -35.6)
- added LED13: 10mA 2.7-3.5V, Diode_SMD:D_0603_1608Metric_Pad1.05x0.95mm_HandSolder, F.Cu at (192.1, -33.0)
- added LED14: 10mA 2.7-3.5V, Diode_SMD:D_0603_1608Metric_Pad1.05x0.95mm_HandSolder, F.Cu at (192.1, -30.4)
- added LED15: 10mA 2.7-3.5V, Diode_SMD:D_0603_1608Metric_Pad1.05x0.95mm_HandSolder, F.Cu at (192.1, -27.8)
- added LED16: 10mA 2.7-3.5V, Diode_SMD:D_0603_1608Metric_Pad1.05x0.95mm_HandSolder, F.Cu at (192.1, -25.2)
- added LED17: 10mA 2.7-3.5V, Diode_SMD:D_0603_1608Metric_Pad1.05x0.95mm_HandSolder, F.Cu at (192.1, -22.6)
- added LED18: 10mA 2.7-3.5V, Diode_SMD:D_0603_1608Metric_Pad1.05x0.95mm_HandSolder, F.Cu at (192.1, -20.0)
- added LED19: 10mA 2.7-3.5V, Diode_SMD:D_0603_1608Metric_Pad1.05x0.95mm_HandSolder, F.Cu at (192.1, -17.4)
- added LED2: 10mA 2.7-3.5V, Diode_SMD:D_0603_1608Metric_Pad1.05x0.95mm_HandSolder, F.Cu at (187.7, -35.6)
- added LED20: 10mA 2.7-3.5V, Diode_SMD:D_0603_1608Metric_Pad1.05x0.95mm_HandSolder, F.Cu at (192.1, -14.8)
- added LED21: 10mA 2.7-3.5V, Diode_SMD:D_0603_1608Metric_Pad1.05x0.95mm_HandSolder, F.Cu at (196.5, -38.1)
- added LED22: 10mA 2.7-3.5V, Diode_SMD:D_0603_1608Metric_Pad1.05x0.95mm_HandSolder, F.Cu at (196.5, -35.6)
- added LED23: 10mA 2.7-3.5V, Diode_SMD:D_0603_1608Metric_Pad1.05x0.95mm_HandSolder, F.Cu at (196.5, -33.0)
- added LED24: 10mA 2.7-3.5V, Diode_SMD:D_0603_1608Metric_Pad1.05x0.95mm_HandSolder, F.Cu at (196.5, -30.4)
- added LED25: 10mA 2.7-3.5V, Diode_SMD:D_0603_1608Metric_Pad1.05x0.95mm_HandSolder, F.Cu at (196.5, -27.8)
- added LED26: 10mA 2.7-3.5V, Diode_SMD:D_0603_1608Metric_Pad1.05x0.95mm_HandSolder, F.Cu at (196.5, -25.2)
- added LED27: 10mA 2.7-3.5V, Diode_SMD:D_0603_1608Metric_Pad1.05x0.95mm_HandSolder, F.Cu at (196.5, -22.6)
- added LED28: 10mA 2.7-3.5V, Diode_SMD:D_0603_1608Metric_Pad1.05x0.95mm_HandSolder, F.Cu at (196.5, -20.0)
- added LED29: 10mA 2.7-3.5V, Diode_SMD:D_0603_1608Metric_Pad1.05x0.95mm_HandSolder, F.Cu at (196.5, -17.4)
- added LED3: 10mA 2.7-3.5V, Diode_SMD:D_0603_1608Metric_Pad1.05x0.95mm_HandSolder, F.Cu at (187.7, -33.0)
- added LED30: 10mA 2.7-3.5V, Diode_SMD:D_0603_1608Metric_Pad1.05x0.95mm_HandSolder, F.Cu at (196.5, -14.8)
- added LED31: 10mA 2.7-3.5V, Diode_SMD:D_0603_1608Metric_Pad1.05x0.95mm_HandSolder, F.Cu at (200.9, -38.1)
- added LED32: 10mA 2.7-3.5V, Diode_SMD:D_0603_1608Metric_Pad1.05x0.95mm_HandSolder, F.Cu at (200.9, -35.6)
- added LED33: 10mA 2.7-3.5V, Diode_SMD:D_0603_1608Metric_Pad1.05x0.95mm_HandSolder, F.Cu at (200.9, -33.0)
- added LED34: 10mA 2.7-3.5V, Diode_SMD:D_0603_1608Metric_Pad1.05x0.95mm_HandSolder, F.Cu at (200.9, -30.4)
- added LED35: 10mA 2.7-3.5V, Diode_SMD:D_0603_1608Metric_Pad1.05x0.95mm_HandSolder, F.Cu at (200.9, -27.8)
- added LED36: 10mA 2.7-3.5V, Diode_SMD:D_0603_1608Metric_Pad1.05x0.95mm_HandSolder, F.Cu at (200.9, -25.2)
- added LED37: 10mA 2.7-3.5V, Diode_SMD:D_0603_1608Metric_Pad1.05x0.95mm_HandSolder, F.Cu at (200.9, -22.6)
- added LED38: 10mA 2.7-3.5V, Diode_SMD:D_0603_1608Metric_Pad1.05x0.95mm_HandSolder, F.Cu at (200.9, -20.0)
- added LED39: 10mA 2.7-3.5V, Diode_SMD:D_0603_1608Metric_Pad1.05x0.95mm_HandSolder, F.Cu at (200.9, -17.4)
- added LED4: 10mA 2.7-3.5V, Diode_SMD:D_0603_1608Metric_Pad1.05x0.95mm_HandSolder, F.Cu at (187.7, -30.4)
- added LED40: 10mA 2.7-3.5V, Diode_SMD:D_0603_1608Metric_Pad1.05x0.95mm_HandSolder, F.Cu at (200.9, -14.8)
- added LED41: 10mA 2.7-3.5V, Diode_SMD:D_0603_1608Metric_Pad1.05x0.95mm_HandSolder, F.Cu at (205.3, -38.1)
- added LED42: 10mA 2.7-3.5V, Diode_SMD:D_0603_1608Metric_Pad1.05x0.95mm_HandSolder, F.Cu at (205.3, -35.6)
- added LED43: 10mA 2.7-3.5V, Diode_SMD:D_0603_1608Metric_Pad1.05x0.95mm_HandSolder, F.Cu at (205.3, -33.0)
- added LED44: 10mA 2.7-3.5V, Diode_SMD:D_0603_1608Metric_Pad1.05x0.95mm_HandSolder, F.Cu at (205.3, -30.4)
- added LED45: 10mA 2.7-3.5V, Diode_SMD:D_0603_1608Metric_Pad1.05x0.95mm_HandSolder, F.Cu at (205.3, -27.8)
- added LED46: 10mA 2.7-3.5V, Diode_SMD:D_0603_1608Metric_Pad1.05x0.95mm_HandSolder, F.Cu at (205.3, -25.2)
- added LED47: 10mA 2.7-3.5V, Diode_SMD:D_0603_1608Metric_Pad1.05x0.95mm_HandSolder, F.Cu at (205.3, -22.6)
- added LED48: 10mA 2.7-3.5V, Diode_SMD:D_0603_1608Metric_Pad1.05x0.95mm_HandSolder, F.Cu at (205.3, -20.0)
- added LED5: 10mA 2.7-3.5V, Diode_SMD:D_0603_1608Metric_Pad1.05x0.95mm_HandSolder, F.Cu at (187.7, -27.8)
- added LED6: 10mA 2.7-3.5V, Diode_SMD:D_0603_1608Metric_Pad1.05x0.95mm_HandSolder, F.Cu at (187.7, -25.2)
- added LED7: 10mA 2.7-3.5V, Diode_SMD:D_0603_1608Metric_Pad1.05x0.95mm_HandSolder, F.Cu at (187.7, -22.6)
- added LED8: 10mA 2.7-3.5V, Diode_SMD:D_0603_1608Metric_Pad1.05x0.95mm_HandSolder, F.Cu at (187.7, -20.0)
- added LED9: 10mA 2.7-3.5V, Diode_SMD:D_0603_1608Metric_Pad1.05x0.95mm_HandSolder, F.Cu at (187.7, -17.4)
- added LIGHTGATE1: Conn_01x03, Connector_JST:JST_XH_B3B-XH-A_1x03_P2.50mm_Vertical, F.Cu at (147.3, 24.6)
- added LOADCELL1: Conn_01x04, Connector_JST:JST_XH_B4B-XH-A_1x04_P2.50mm_Vertical, F.Cu at (161.7, 11.2)
- added MOUSE1: ~, custom:PMW3360_breakout, F.Cu at (-86.0, 0.00)
- added MOUSE2: ~, custom:PMW3360_breakout, F.Cu at (86.0, 0.00)
- added MOUSE_FPC1: FC10-S08FCT-00, EasyEDA:FPC-SMD_8P-P1.00_DEALON_FC10-S08FCT-00, F.Cu at (165.4, 18.2)
- added MOUSE_FPC2: FC10-S08FCT-00, EasyEDA:FPC-SMD_8P-P1.00_DEALON_FC10-S08FCT-00, F.Cu at (165.4, 25.7)
- added R100: 240R, PCM_Resistor_SMD_AKL:R_0805_2012Metric_Pad1.15x1.40mm_HandSolder, F.Cu at (207.1, -62.1)
- added R101: 240R, PCM_Resistor_SMD_AKL:R_0805_2012Metric_Pad1.15x1.40mm_HandSolder, F.Cu at (207.1, -59.1)
- added R102: 240R, PCM_Resistor_SMD_AKL:R_0805_2012Metric_Pad1.15x1.40mm_HandSolder, F.Cu at (207.1, -56.1)
- added R103: 240R, PCM_Resistor_SMD_AKL:R_0805_2012Metric_Pad1.15x1.40mm_HandSolder, F.Cu at (207.1, -53.0)
- added R104: 240R, PCM_Resistor_SMD_AKL:R_0805_2012Metric_Pad1.15x1.40mm_HandSolder, F.Cu at (207.1, -50.0)
- added R105: 240R, PCM_Resistor_SMD_AKL:R_0805_2012Metric_Pad1.15x1.40mm_HandSolder, F.Cu at (207.1, -47.0)
- added R106: 240R, PCM_Resistor_SMD_AKL:R_0805_2012Metric_Pad1.15x1.40mm_HandSolder, F.Cu at (207.1, -44.0)
- added R107: 240R, PCM_Resistor_SMD_AKL:R_0805_2012Metric_Pad1.15x1.40mm_HandSolder, F.Cu at (207.1, -41.0)
- added R108: 240R, PCM_Resistor_SMD_AKL:R_0805_2012Metric_Pad1.15x1.40mm_HandSolder, F.Cu at (211.9, -62.1)
- added R109: 240R, PCM_Resistor_SMD_AKL:R_0805_2012Metric_Pad1.15x1.40mm_HandSolder, F.Cu at (211.9, -59.1)
- added R110: 240R, PCM_Resistor_SMD_AKL:R_0805_2012Metric_Pad1.15x1.40mm_HandSolder, F.Cu at (211.9, -56.1)
- added R111: 240R, PCM_Resistor_SMD_AKL:R_0805_2012Metric_Pad1.15x1.40mm_HandSolder, F.Cu at (211.9, -53.0)
- added R112: 240R, PCM_Resistor_SMD_AKL:R_0805_2012Metric_Pad1.15x1.40mm_HandSolder, F.Cu at (211.9, -50.0)
- added R113: 240R, PCM_Resistor_SMD_AKL:R_0805_2012Metric_Pad1.15x1.40mm_HandSolder, F.Cu at (211.9, -47.0)
- added R114: 240R, PCM_Resistor_SMD_AKL:R_0805_2012Metric_Pad1.15x1.40mm_HandSolder, F.Cu at (211.9, -44.0)
- added R115: 240R, PCM_Resistor_SMD_AKL:R_0805_2012Metric_Pad1.15x1.40mm_HandSolder, F.Cu at (211.9, -41.0)
- added R53: DNP, PCM_Resistor_SMD_AKL:R_0805_2012Metric_Pad1.15x1.40mm_HandSolder, F.Cu at (146.2, 13.6)
- added R54: 0R, PCM_Resistor_SMD_AKL:R_0805_2012Metric_Pad1.15x1.40mm_HandSolder, F.Cu at (146.2, 16.7)
- added R55: DNP, PCM_Resistor_SMD_AKL:R_0805_2012Metric_Pad1.15x1.40mm_HandSolder, F.Cu at (146.2, 19.7)
- added R56: 0R, PCM_Resistor_SMD_AKL:R_0805_2012Metric_Pad1.15x1.40mm_HandSolder, F.Cu at (151.0, 1.54)
- added R57: DNP, PCM_Resistor_SMD_AKL:R_0805_2012Metric_Pad1.15x1.40mm_HandSolder, F.Cu at (151.0, 4.57)
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Connections:
- net +12V renamed VCC
- net /MISO renamed /SPI0.MISO
- net /MOSI renamed /SPI0.MOSI
- net /SCL renamed /I2C0.SCL
- net /SCLK renamed /SPI0.SCLK
- net /SDA renamed /I2C0.SDA
- ADC1 pad 7: /DRV4_IPROPI -> /GATE
- ADC2 pad 2: /ADC_INT -> /ADC_INT2
- ADC2 pad 4: /DRV5_IPROPI -> /DRV4_IPROPI
- ADC2 pad 5: unconnected-(ADC2-AIN1-Pad5) -> /DRV5_IPROPI
- ADC2 pad 6: unconnected-(ADC2-AIN2-Pad6) -> /LOADCELL_A+
- ADC2 pad 7: unconnected-(ADC2-AIN3-Pad7) -> /LOADCELL_A-
- PR1 pad 1: +3.3V -> +3V3
- PR10 pad 1: +3.3V -> +3V3
- PR11 pad 1: +3.3V -> +3V3
- PR12 pad 1: +3.3V -> +3V3
- PR13 pad 1: +3.3V -> +3V3
- PR14 pad 1: +3.3V -> +3V3
- PR15 pad 1: +3.3V -> +3V3
- PR16 pad 1: +3.3V -> +3V3
- PR17 pad 1: +3.3V -> +3V3
- PR18 pad 1: +3.3V -> +3V3
- PR19 pad 1: +3.3V -> +3V3
- PR2 pad 1: +3.3V -> +3V3
- PR20 pad 1: +3.3V -> +3V3
- PR21 pad 1: +3.3V -> +3V3
- PR22 pad 1: +3.3V -> +3V3
- PR23 pad 1: +3.3V -> +3V3
- PR24 pad 1: +3.3V -> +3V3
- PR25 pad 1: +3.3V -> +3V3
- PR26 pad 1: +3.3V -> +3V3
- PR27 pad 1: +3.3V -> +3V3
- PR28 pad 1: +3.3V -> +3V3
- PR29 pad 1: +3.3V -> +3V3
- PR3 pad 1: +3.3V -> +3V3
- PR30 pad 1: +3.3V -> +3V3
- PR31 pad 1: +3.3V -> +3V3
- PR32 pad 1: +3.3V -> +3V3
- PR33 pad 1: +3.3V -> +3V3
- PR34 pad 1: +3.3V -> +3V3
- PR35 pad 1: +3.3V -> +3V3
- PR36 pad 1: +3.3V -> +3V3
- PR37 pad 1: +3.3V -> +3V3
- PR38 pad 1: +3.3V -> +3V3
- PR39 pad 1: +3.3V -> +3V3
- PR4 pad 1: +3.3V -> +3V3
- PR40 pad 1: +3.3V -> +3V3
- PR41 pad 1: +3.3V -> +3V3
- PR42 pad 1: +3.3V -> +3V3
- PR43 pad 1: +3.3V -> +3V3
- PR44 pad 1: +3.3V -> +3V3
- PR45 pad 1: +3.3V -> +3V3
- PR46 pad 1: +3.3V -> +3V3
- PR47 pad 1: +3.3V -> +3V3
- PR48 pad 1: +3.3V -> +3V3
- PR5 pad 1: +3.3V -> +3V3
- PR6 pad 1: +3.3V -> +3V3
- PR7 pad 1: +3.3V -> +3V3
- PR8 pad 1: +3.3V -> +3V3
- PR9 pad 1: +3.3V -> +3V3
- U1 pad 10: unconnected-(U1-GPIO7-Pad10) -> /DRV1_IN2
- U1 pad 11: unconnected-(U1-GPIO8-Pad11) -> /DRV2_IN1
- U1 pad 12: unconnected-(U1-GPIO9-Pad12) -> /DRV2_IN2
- U1 pad 14: unconnected-(U1-GPIO10-Pad14) -> /DRV3_IN1
- U1 pad 15: unconnected-(U1-GPIO11-Pad15) -> /DRV3_IN2
- U1 pad 16: unconnected-(U1-GPIO12-Pad16) -> /DRV4_IN1
- U1 pad 17: unconnected-(U1-GPIO13-Pad17) -> /DRV4_IN2
- U1 pad 19: unconnected-(U1-GPIO14-Pad19) -> /DRV5_IN1
- U1 pad 20: unconnected-(U1-GPIO15-Pad20) -> /DRV5_IN2
- U1 pad 21: unconnected-(U1-GPIO16-Pad21) -> /TX0
- U1 pad 22: unconnected-(U1-GPIO17-Pad22) -> /RX0
- U1 pad 24: unconnected-(U1-GPIO18-Pad24) -> /KICK
- U1 pad 25: unconnected-(U1-GPIO19-Pad25) -> /DMUX1_INT
- U1 pad 26: unconnected-(U1-GPIO20-Pad26) -> /DMUX_RESET
- U1 pad 27: unconnected-(U1-GPIO21-Pad27) -> /DMUX_SCS
- U1 pad 29: unconnected-(U1-GPIO22-Pad29) -> /MOUSE1_SCS
- U1 pad 30: unconnected-(U1-RUN-Pad30) -> /RUN
- U1 pad 31: MUX1_COM -> AMUX1_COM
- U1 pad 32: MUX2_COM -> AMUX2_COM
- U1 pad 34: MUX3_COM -> AMUX3_COM
- U1 pad 36: +3V3 -> unconnected-(U1-3V3-Pad36)
- U1 pad 37: unconnected-(U1-3V3_EN-Pad37) -> /EN
- U1 pad 39: unconnected-(U1-VSYS-Pad39) -> +5V
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Other:
- board size 64 x 63.5 mm -> 218 x 205.9 mm
- copper layers 2 -> 4

Commit message: cleaned up bottom plate schematic and added explanations of design decisions. Please read.
Parts:
- added GATE_LED1: Conn_01x02, Connector_JST:JST_XH_B2B-XH-A_1x02_P2.50mm_Vertical, F.Cu at (111.8, -62.5)
- added PWR2: XT30-F, Connector_AMASS:AMASS_XT30U-F_1x02_P5.0mm_Vertical, F.Cu at (19.5, 17.0)
- added R67: 4.7k, PCM_Resistor_SMD_AKL:R_0805_2012Metric_Pad1.15x1.40mm_HandSolder, F.Cu at (1.90, 1.01)
- C2: value 22uF -> 1uF
- C3: value 1uF -> 22uF
- LED1: value 10mA 2.7-3.5V -> 2.8-3.4V 1400mcd@20mA; footprint Diode_SMD:D_0603_1608Metric_Pad1.05x0.95mm_HandSolder -> Diode_SMD:D_0805_2012Metric_Pad1.15x1.40mm_HandSolder; moved to B.Cu
- LED10, LED11, LED12, LED13, LED14, LED15, LED16, LED17, LED18, LED19, LED2, LED20, LED21, LED22, LED23, LED24, LED25, LED26, LED27, LED28, LED29, LED3, LED30, LED31, LED32, LED33, LED34, LED35, LED36, LED37, LED38, LED39, LED4, LED40, LED41, LED42, LED43, LED44, LED45, LED46, LED47, LED48, LED5, LED6, LED7, LED8, LED9: value 10mA 2.7-3.5V -> 2.8-3.4V 1400mcd@20mA; footprint Diode_SMD:D_0603_1608Metric_Pad1.05x0.95mm_HandSolder -> Diode_SMD:D_0805_2012Metric_Pad1.15x1.40mm_HandSolder
- R10, R12, R14, R16, R18, R2, R20, R22, R24, R26, R28, R30, R32, R34, R36, R38, R4, R40, R42, R44, R46, R48, R6, R8: value 4.7k -> 220R
- R100, R102, R104, R106, R108, R110, R112, R114, R70, R72, R74, R76, R78, R80, R82, R84, R86, R88, R90, R92, R94, R96, R98: value 240R -> 220R
- R101, R103, R105, R107, R109, R111, R113, R69, R71, R73, R75, R77, R79, R81, R83, R85, R87, R89, R91, R93, R95, R97, R99: value 240R -> 4.7k
- R68: value 240R -> 220R; moved to B.Cu
- U1: footprint RP-Pico Libraries:RPi_Pico_SMD_TH -> RP-Pico Libraries:RPi_Pico_SMD_TH_USBC_cable_cutout
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Connections:
- net AMUX_EN renamed /AMUX_EN
- net MUX_S0 renamed /AMUX_S0
- net MUX_S1 renamed /AMUX_S1
- net MUX_S2 renamed /AMUX_S2
- net MUX_S3 renamed /AMUX_S3
- AMUX1 pad 16: /line sensors/PR16 -> /line sensor array 1/LS16
- AMUX1 pad 17: /line sensors/PR15 -> /line sensor array 1/LS15
- AMUX1 pad 18: /line sensors/PR14 -> /line sensor array 1/LS14
- AMUX1 pad 19: /line sensors/PR13 -> /line sensor array 1/LS13
- AMUX1 pad 2: /line sensors/PR8 -> /line sensor array 1/LS8
- AMUX1 pad 20: /line sensors/PR12 -> /line sensor array 1/LS12
- AMUX1 pad 21: /line sensors/PR11 -> /line sensor array 1/LS11
- AMUX1 pad 22: /line sensors/PR10 -> /line sensor array 1/LS10
- AMUX1 pad 23: /line sensors/PR9 -> /line sensor array 1/LS9
- AMUX1 pad 3: /line sensors/PR7 -> /line sensor array 1/LS7
- AMUX1 pad 4: /line sensors/PR6 -> /line sensor array 1/LS6
- AMUX1 pad 5: /line sensors/PR5 -> /line sensor array 1/LS5
- AMUX1 pad 6: /line sensors/PR4 -> /line sensor array 1/LS4
- AMUX1 pad 7: /line sensors/PR3 -> /line sensor array 1/LS3
- AMUX1 pad 8: /line sensors/PR2 -> /line sensor array 1/LS2
- AMUX1 pad 9: /line sensors/PR1 -> /line sensor array 1/LS1
- AMUX2 pad 16: /line sensors/PR32 -> /line sensor array 2/LS16
- AMUX2 pad 17: /line sensors/PR31 -> /line sensor array 2/LS15
- AMUX2 pad 18: /line sensors/PR30 -> /line sensor array 2/LS14
- AMUX2 pad 19: /line sensors/PR29 -> /line sensor array 2/LS13
- AMUX2 pad 2: /line sensors/PR24 -> /line sensor array 2/LS8
- AMUX2 pad 20: /line sensors/PR28 -> /line sensor array 2/LS12
- AMUX2 pad 21: /line sensors/PR27 -> /line sensor array 2/LS11
- AMUX2 pad 22: /line sensors/PR26 -> /line sensor array 2/LS10
- AMUX2 pad 23: /line sensors/PR25 -> /line sensor array 2/LS9
- AMUX2 pad 3: /line sensors/PR23 -> /line sensor array 2/LS7
- AMUX2 pad 4: /line sensors/PR22 -> /line sensor array 2/LS6
- AMUX2 pad 5: /line sensors/PR21 -> /line sensor array 2/LS5
- AMUX2 pad 6: /line sensors/PR20 -> /line sensor array 2/LS4
- AMUX2 pad 7: /line sensors/PR19 -> /line sensor array 2/LS3
- AMUX2 pad 8: /line sensors/PR18 -> /line sensor array 2/LS2
- AMUX2 pad 9: /line sensors/PR17 -> /line sensor array 2/LS1
- AMUX3 pad 16: /line sensors/PR48 -> /line sensor array 3/LS16
- AMUX3 pad 17: /line sensors/PR47 -> /line sensor array 3/LS15
- AMUX3 pad 18: /line sensors/PR46 -> /line sensor array 3/LS14
- AMUX3 pad 19: /line sensors/PR45 -> /line sensor array 3/LS13
- AMUX3 pad 2: /line sensors/PR40 -> /line sensor array 3/LS8
- AMUX3 pad 20: /line sensors/PR44 -> /line sensor array 3/LS12
- AMUX3 pad 21: /line sensors/PR43 -> /line sensor array 3/LS11
- AMUX3 pad 22: /line sensors/PR42 -> /line sensor array 3/LS10
- AMUX3 pad 23: /line sensors/PR41 -> /line sensor array 3/LS9
- AMUX3 pad 3: /line sensors/PR39 -> /line sensor array 3/LS7
- AMUX3 pad 4: /line sensors/PR38 -> /line sensor array 3/LS6
- AMUX3 pad 5: /line sensors/PR37 -> /line sensor array 3/LS5
- AMUX3 pad 6: /line sensors/PR36 -> /line sensor array 3/LS4
- AMUX3 pad 7: /line sensors/PR35 -> /line sensor array 3/LS3
- AMUX3 pad 8: /line sensors/PR34 -> /line sensor array 3/LS2
- AMUX3 pad 9: /line sensors/PR33 -> /line sensor array 3/LS1
- C2 pad 1: GND -> unconnected-(C2-Pad1)
- C2 pad 2: unconnected-(C2-Pad2) -> +5V
- C3 pad 1: unconnected-(C3-Pad1) -> GND
- C3 pad 2: +5V -> unconnected-(C3-Pad2)
- DMUX1 pad 1: /ADC_INT1 -> /DRV1_OFF
- DMUX1 pad 2: /ADC_INT2 -> /DRV1_NSLEEP
- DMUX1 pad 21: /DRV5_NFAULT -> /MOUSE1_SCS
- DMUX1 pad 22: /DMUX2_INT -> /MOUSE2_SCS
- DMUX1 pad 3: /MOUSE1_MOT -> /DRV2_OFF
- DMUX1 pad 4: /MOUSE2_MOT -> /DRV2_NSLEEP
- DMUX1 pad 5: /DRV1_NFAULT -> /DRV3_OFF
- DMUX1 pad 6: /DRV2_NFAULT -> /DRV3_NSLEEP
- DMUX1 pad 7: /DRV3_NFAULT -> /DRV4_OFF
- DMUX1 pad 8: /DRV4_NFAULT -> /DRV4_NSLEEP
- DMUX2 pad 1: /DRV1_OFF -> /DRV1_NFAULT
- DMUX2 pad 2: /DRV1_NSLEEP -> /DRV2_NFAULT
- DMUX2 pad 21: /DRV5_OFF -> /DRV1_SCS
- DMUX2 pad 22: /DRV5_NSLEEP -> /DRV2_SCS
- DMUX2 pad 23: /DRV1_SCS -> /DRV3_SCS
- DMUX2 pad 24: /DRV2_SCS -> /DRV4_SCS
- DMUX2 pad 25: /DRV3_SCS -> /DRV5_SCS
- DMUX2 pad 26: /DRV4_SCS -> /DRV5_OFF
- DMUX2 pad 27: /DRV5_SCS -> /DRV5_NSLEEP
- DMUX2 pad 3: /DRV2_OFF -> /DRV3_NFAULT
- DMUX2 pad 4: /DRV2_NSLEEP -> /DRV4_NFAULT
- DMUX2 pad 5: /DRV3_OFF -> /DRV5_NFAULT
- DMUX2 pad 6: /DRV3_NSLEEP -> /ADC_INT1
- DMUX2 pad 7: /DRV4_OFF -> /ADC_INT2
- DMUX2 pad 8: /DRV4_NSLEEP -> /DMUX2_INT
- LED1 pad 1: GND -> Net-(LED1-K)
- LED1 pad 2: Net-(LED1-A) -> +5V
- LED10 pad 1: GND -> Net-(LED10-K)
- LED10 pad 2: Net-(LED10-A) -> +5V
- LED11 pad 1: GND -> Net-(LED11-K)
- LED11 pad 2: Net-(LED11-A) -> +5V
- LED12 pad 1: GND -> Net-(LED12-K)
- LED12 pad 2: Net-(LED12-A) -> +5V
- LED13 pad 1: GND -> Net-(LED13-K)
- LED13 pad 2: Net-(LED13-A) -> +5V
- LED14 pad 1: GND -> Net-(LED14-K)
- LED14 pad 2: Net-(LED14-A) -> +5V
- LED15 pad 1: GND -> Net-(LED15-K)
- LED15 pad 2: Net-(LED15-A) -> +5V
- LED16 pad 1: GND -> Net-(LED16-K)
- LED16 pad 2: Net-(LED16-A) -> +5V
- LED17 pad 1: GND -> Net-(LED17-K)
- LED17 pad 2: Net-(LED17-A) -> +5V
- LED18 pad 1: GND -> Net-(LED18-K)
- LED18 pad 2: Net-(LED18-A) -> +5V
- LED19 pad 1: GND -> Net-(LED19-K)
- LED19 pad 2: Net-(LED19-A) -> +5V
- LED2 pad 1: GND -> Net-(LED2-K)
- LED2 pad 2: Net-(LED2-A) -> +5V
- LED20 pad 1: GND -> Net-(LED20-K)
- LED20 pad 2: Net-(LED20-A) -> +5V
- LED21 pad 1: GND -> Net-(LED21-K)
- LED21 pad 2: Net-(LED21-A) -> +5V
- LED22 pad 1: GND -> Net-(LED22-K)
- LED22 pad 2: Net-(LED22-A) -> +5V
- LED23 pad 1: GND -> Net-(LED23-K)
- LED23 pad 2: Net-(LED23-A) -> +5V
- LED24 pad 1: GND -> Net-(LED24-K)
- LED24 pad 2: Net-(LED24-A) -> +5V
- LED25 pad 1: GND -> Net-(LED25-K)
- LED25 pad 2: Net-(LED25-A) -> +5V
- LED26 pad 1: GND -> Net-(LED26-K)
- LED26 pad 2: Net-(LED26-A) -> +5V
- LED27 pad 1: GND -> Net-(LED27-K)
- LED27 pad 2: Net-(LED27-A) -> +5V
- LED28 pad 1: GND -> Net-(LED28-K)
- LED28 pad 2: Net-(LED28-A) -> +5V
- LED29 pad 1: GND -> Net-(LED29-K)
- LED29 pad 2: Net-(LED29-A) -> +5V
- LED3 pad 1: GND -> Net-(LED3-K)
- LED3 pad 2: Net-(LED3-A) -> +5V
- LED30 pad 1: GND -> Net-(LED30-K)
- LED30 pad 2: Net-(LED30-A) -> +5V
- LED31 pad 1: GND -> Net-(LED31-K)
- LED31 pad 2: Net-(LED31-A) -> +5V
- LED32 pad 1: GND -> Net-(LED32-K)
- LED32 pad 2: Net-(LED32-A) -> +5V
- LED33 pad 1: GND -> Net-(LED33-K)
- LED33 pad 2: Net-(LED33-A) -> +5V
- LED34 pad 1: GND -> Net-(LED34-K)
- LED34 pad 2: Net-(LED34-A) -> +5V
- LED35 pad 1: GND -> Net-(LED35-K)
- LED35 pad 2: Net-(LED35-A) -> +5V
- LED36 pad 1: GND -> Net-(LED36-K)
- LED36 pad 2: Net-(LED36-A) -> +5V
- LED37 pad 1: GND -> Net-(LED37-K)
- LED37 pad 2: Net-(LED37-A) -> +5V
- LED38 pad 1: GND -> Net-(LED38-K)
- LED38 pad 2: Net-(LED38-A) -> +5V
- LED39 pad 1: GND -> Net-(LED39-K)
- LED39 pad 2: Net-(LED39-A) -> +5V
- LED4 pad 1: GND -> Net-(LED4-K)
- LED4 pad 2: Net-(LED4-A) -> +5V
- LED40 pad 1: GND -> Net-(LED40-K)
- LED40 pad 2: Net-(LED40-A) -> +5V
- LED41 pad 1: GND -> Net-(LED41-K)
- LED41 pad 2: Net-(LED41-A) -> +5V
- LED42 pad 1: GND -> Net-(LED42-K)
- LED42 pad 2: Net-(LED42-A) -> +5V
- LED43 pad 1: GND -> Net-(LED43-K)
- LED43 pad 2: Net-(LED43-A) -> +5V
- LED44 pad 1: GND -> Net-(LED44-K)
- LED44 pad 2: Net-(LED44-A) -> +5V
- LED45 pad 1: GND -> Net-(LED45-K)
- LED45 pad 2: Net-(LED45-A) -> +5V
- LED46 pad 1: GND -> Net-(LED46-K)
- LED46 pad 2: Net-(LED46-A) -> +5V
- LED47 pad 1: GND -> Net-(LED47-K)
- LED47 pad 2: Net-(LED47-A) -> +5V
- LED48 pad 1: GND -> Net-(LED48-K)
- LED48 pad 2: Net-(LED48-A) -> +5V
- LED5 pad 1: GND -> Net-(LED5-K)
- LED5 pad 2: Net-(LED5-A) -> +5V
- LED6 pad 1: GND -> Net-(LED6-K)
- LED6 pad 2: Net-(LED6-A) -> +5V
- LED7 pad 1: GND -> Net-(LED7-K)
- LED7 pad 2: Net-(LED7-A) -> +5V
- LED8 pad 1: GND -> Net-(LED8-K)
- LED8 pad 2: Net-(LED8-A) -> +5V
- LED9 pad 1: GND -> Net-(LED9-K)
- LED9 pad 2: Net-(LED9-A) -> +5V
- PR1 pad 2: /line sensors/PR1 -> /line sensor array 1/LS2
- PR10 pad 2: /line sensors/PR10 -> /line sensor array 1/LS10
- PR11 pad 2: /line sensors/PR11 -> /line sensor array 1/LS15
- PR12 pad 2: /line sensors/PR12 -> /line sensor array 1/LS16
- PR13 pad 2: /line sensors/PR13 -> /line sensor array 1/LS11
- PR14 pad 2: /line sensors/PR14 -> /line sensor array 1/LS12
- PR15 pad 2: /line sensors/PR15 -> /line sensor array 1/LS13
- PR16 pad 2: /line sensors/PR16 -> /line sensor array 1/LS14
- PR17 pad 2: /line sensors/PR17 -> /line sensor array 2/LS2
- PR18 pad 2: /line sensors/PR18 -> /line sensor array 2/LS1
- PR19 pad 2: /line sensors/PR19 -> /line sensor array 2/LS8
- PR2 pad 2: /line sensors/PR2 -> /line sensor array 1/LS1
- PR20 pad 2: /line sensors/PR20 -> /line sensor array 2/LS7
- PR21 pad 2: /line sensors/PR21 -> /line sensor array 2/LS4
- PR22 pad 2: /line sensors/PR22 -> /line sensor array 2/LS3
- PR23 pad 2: /line sensors/PR23 -> /line sensor array 2/LS5
- PR24 pad 2: /line sensors/PR24 -> /line sensor array 2/LS6
- PR25 pad 2: /line sensors/PR25 -> /line sensor array 2/LS9
- PR26 pad 2: /line sensors/PR26 -> /line sensor array 2/LS10
- PR27 pad 2: /line sensors/PR27 -> /line sensor array 2/LS15
- PR28 pad 2: /line sensors/PR28 -> /line sensor array 2/LS16
- PR29 pad 2: /line sensors/PR29 -> /line sensor array 2/LS11
- PR3 pad 2: /line sensors/PR3 -> /line sensor array 1/LS8
- PR30 pad 2: /line sensors/PR30 -> /line sensor array 2/LS12
- PR31 pad 2: /line sensors/PR31 -> /line sensor array 2/LS13
- PR32 pad 2: /line sensors/PR32 -> /line sensor array 2/LS14
- PR33 pad 2: /line sensors/PR33 -> /line sensor array 3/LS2
- PR34 pad 2: /line sensors/PR34 -> /line sensor array 3/LS1
- PR35 pad 2: /line sensors/PR35 -> /line sensor array 3/LS8
- PR36 pad 2: /line sensors/PR36 -> /line sensor array 3/LS7
- PR37 pad 2: /line sensors/PR37 -> /line sensor array 3/LS4
- PR38 pad 2: /line sensors/PR38 -> /line sensor array 3/LS3
- PR39 pad 2: /line sensors/PR39 -> /line sensor array 3/LS5
- PR4 pad 2: /line sensors/PR4 -> /line sensor array 1/LS7
- PR40 pad 2: /line sensors/PR40 -> /line sensor array 3/LS6
- PR41 pad 2: /line sensors/PR41 -> /line sensor array 3/LS9
- PR42 pad 2: /line sensors/PR42 -> /line sensor array 3/LS10
- PR43 pad 2: /line sensors/PR43 -> /line sensor array 3/LS15
- PR44 pad 2: /line sensors/PR44 -> /line sensor array 3/LS16
- PR45 pad 2: /line sensors/PR45 -> /line sensor array 3/LS11
- PR46 pad 2: /line sensors/PR46 -> /line sensor array 3/LS12
- PR47 pad 2: /line sensors/PR47 -> /line sensor array 3/LS13
- PR48 pad 2: /line sensors/PR48 -> /line sensor array 3/LS14
- PR5 pad 2: /line sensors/PR5 -> /line sensor array 1/LS4
- PR6 pad 2: /line sensors/PR6 -> /line sensor array 1/LS3
- PR7 pad 2: /line sensors/PR7 -> /line sensor array 1/LS5
- PR8 pad 2: /line sensors/PR8 -> /line sensor array 1/LS6
- PR9 pad 2: /line sensors/PR9 -> /line sensor array 1/LS9
- R1 pad 1: /line sensors/PR1 -> /line sensor array 1/LS2
- R10 pad 1: /line sensors/PR10 -> GND
- R10 pad 2: GND -> Net-(LED5-K)
- R100 pad 1: Net-(LED33-A) -> GND
- R100 pad 2: +5V -> Net-(LED41-K)
- R101 pad 1: Net-(LED34-A) -> /line sensor array 3/LS10
- R101 pad 2: +5V -> GND
- R102 pad 1: Net-(LED35-A) -> GND
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Other:
- board text added: "+"
- board text added: "-"

Commit message: cleaned up bottom plate schematic numbering
Parts:
- LED10, LED11, LED12, LED13, LED14, LED15, LED16, LED17, LED18, LED19, LED2, LED20, LED21, LED22, LED23, LED24, LED25, LED26, LED27, LED28, LED29, LED3, LED30, LED31, LED32, LED33, LED34, LED35, LED36, LED37, LED38, LED39, LED4, LED40, LED41, LED42, LED43, LED44, LED45, LED46, LED47, LED48, LED5, LED6, LED7, LED8, LED9, PR1, PR10, PR11, PR12, PR13, PR14, PR15, PR16, PR17, PR18, PR19, PR2, PR20, PR21, PR22, PR23, PR24, PR25, PR26, PR27, PR28, PR29, PR3, PR30, PR31, PR32, PR33, PR34, PR35, PR36, PR37, PR38, PR39, PR4, PR40, PR41, PR42, PR43, PR44, PR45, PR46, PR47, PR48, PR5, PR6, PR7, PR8, PR9, R1, R10, R100, R101, R102, R103, R104, R105, R106, R107, R108, R109, R11, R110, R111, R112, R113, R114, R115, R12, R13, R14, R15, R16, R17, R18, R19, R2, R20, R21, R22, R23, R24, R25, R26, R27, R28, R29, R3, R30, R31, R32, R33, R34, R35, R36, R37, R38, R39, R4, R40, R41, R42, R43, R44, R45, R46, R47, R48, R5, R6, R67, R69, R7, R70, R71, R72, R73, R74, R75, R76, R77, R78, R79, R8, R80, R81, R82, R83, R84, R85, R86, R87, R88, R89, R9, R90, R91, R92, R93, R94, R95, R96, R97, R98, R99: moved to B.Cu
- moved R67 251.6 mm to (253.0, 16.5), turned to 180 degrees
- moved PR1 237.3 mm to (1.00, -64.2), turned to -90 degrees
- moved R1 236.5 mm to (1.00, -60.5), turned to -90 degrees
- moved LED1 235.3 mm to (-1.00, -64.2), turned to 90 degrees
- moved R2 201.6 mm to (-1.00, -60.5), turned to 90 degrees
- moved LED10 163.0 mm to (337.3, 50.0)
- moved LED4 155.8 mm to (314.2, 60.5)
- moved R19 141.5 mm to (333.5, 52.0), turned to 180 degrees
- moved R20 140.2 mm to (333.5, 50.0)
- moved LED8 136.9 mm to (301.5, 56.0)
- moved LED7 133.8 mm to (301.2, 48.2)
- moved LED5 132.2 mm to (301.4, 39.8)
- moved R7 128.2 mm to (310.5, 62.5), turned to 180 degrees
- moved LED6 126.8 mm to (301.2, 31.2)
- moved R8 126.8 mm to (310.5, 60.5)
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Routing:
- net GND: track 0.00 -> 96.0 mm
- net /line sensor array 2/LS8: track 0.00 -> 1.98 mm
- net /line sensor array 2/LS7: track 0.00 -> 1.98 mm
- net /line sensor array 2/LS6: track 0.00 -> 1.98 mm
- net /line sensor array 2/LS5: track 0.00 -> 1.98 mm
- net /line sensor array 2/LS4: track 0.00 -> 1.98 mm
- net /line sensor array 2/LS3: track 0.00 -> 1.98 mm
- net /line sensor array 2/LS1: track 0.00 -> 1.98 mm
- net /line sensor array 1/LS9: track 0.00 -> 1.98 mm
- net /line sensor array 1/LS8: track 0.00 -> 1.98 mm
- net /line sensor array 1/LS7: track 0.00 -> 1.98 mm
- net /line sensor array 1/LS5: track 0.00 -> 1.98 mm
- net /line sensor array 1/LS4: track 0.00 -> 1.98 mm
- net /line sensor array 1/LS3: track 0.00 -> 1.98 mm
- net /line sensor array 1/LS16: track 0.00 -> 1.98 mm
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
Commit message: fixed non convention following of kicker pcb
Parts:
- removed the R1 at (1.00, -60.5)
- removed the R10 at (297.6, 39.8)
- removed R100, R102, R104, R106, R108, R110, R112, R114: 220R, PCM_Resistor_SMD_AKL:R_0805_2012Metric_Pad1.15x1.40mm_HandSolder
- removed R101, R103, R105, R107, R109, R111, R113, R99: 4.7k, PCM_Resistor_SMD_AKL:R_0805_2012Metric_Pad1.15x1.40mm_HandSolder
- removed the R11 at (297.5, 33.2)
- removed R115: 240R, PCM_Resistor_SMD_AKL:R_0805_2012Metric_Pad1.15x1.40mm_HandSolder
- removed the R12 at (297.5, 31.2)
- removed the R15 at (297.8, 58.0)
- removed the R16 at (297.8, 56.0)
- removed the R17 at (264.8, -1.75)
- removed the R18 at (264.8, -3.75)
- removed the R2 at (-1.00, -60.5)
- removed the R3 at (297.6, 17.2)
- removed the R35 at (256.3, 18.8)
- removed the R36 at (256.3, 16.8)
- removed the R37 at (256.3, 21.0)
- removed the R38 at (256.3, 19.0)
- removed the R39 at (256.3, 23.2)
- removed the R4 at (297.6, 15.2)
- removed the R40 at (256.3, 21.2)
- removed the R41 at (256.3, 25.5)
- removed the R42 at (256.3, 23.5)
- removed the R43 at (256.3, 27.8)
- removed the R44 at (256.3, 25.8)
- removed the R45 at (256.3, 30.0)
- removed the R46 at (256.3, 28.0)
- removed the R47 at (256.3, 32.2)
- removed the R48 at (256.3, 30.2)
- removed the R49 at (146.2, 1.54)
- removed the R5 at (255.5, 51.8)
- removed the R50 at (146.2, 4.57)
- removed the R6 at (255.5, 49.8)
- removed the R7 at (310.5, 62.5)
- removed the R8 at (310.5, 60.5)
- removed the R9 at (297.6, 41.8)
- added FH1: XF-506P, EasyEDA:FUSE-TH_XF-506P, F.Cu at (17.5, 13.0)
- added H1: MountingHole_Pad, MountingHole:MountingHole_2.2mm_M2_Pad_Via, F.Cu at (-62.2, -42.4)
- added H10: MountingHole_Pad, MountingHole:MountingHole_2.2mm_M2_Pad_Via, F.Cu at (5.95, -35.7)
- added H11: MountingHole_Pad, MountingHole:MountingHole_2.2mm_M2_Pad_Via, F.Cu at (-45.0, -82.5)
- added H12: MountingHole_Pad, MountingHole:MountingHole_2.2mm_M2_Pad_Via, F.Cu at (45.0, -82.5)
- added H13: MountingHole_Pad, MountingHole:MountingHole_2.2mm_M2_Pad_Via, F.Cu at (82.0, -48.0)
- added H14: MountingHole_Pad, MountingHole:MountingHole_2.2mm_M2_Pad_Via, F.Cu at (82.0, 48.0)
- added H15: MountingHole_Pad, MountingHole:MountingHole_2.2mm_M2_Pad_Via, F.Cu at (45.0, 91.0)
- added H16: MountingHole_Pad, MountingHole:MountingHole_2.2mm_M2_Pad_Via, F.Cu at (-45.0, 91.0)
- added H17: MountingHole_Pad, MountingHole:MountingHole_2.2mm_M2_Pad_Via, F.Cu at (-82.0, 48.0)
- added H18: MountingHole_Pad, MountingHole:MountingHole_2.2mm_M2_Pad_Via, F.Cu at (-82.0, -48.0)
- added H2: MountingHole_Pad, MountingHole:MountingHole_2.2mm_M2_Pad_Via, F.Cu at (-42.4, -62.2)
- added H3: MountingHole_Pad, MountingHole:MountingHole_2.2mm_M2_Pad_Via, F.Cu at (42.4, -62.2)
- added H4: MountingHole_Pad, MountingHole:MountingHole_2.2mm_M2_Pad_Via, F.Cu at (62.2, -42.4)
- added H5: MountingHole_Pad, MountingHole:MountingHole_2.2mm_M2_Pad_Via, F.Cu at (62.2, 42.4)
- added H6: MountingHole_Pad, MountingHole:MountingHole_2.2mm_M2_Pad_Via, F.Cu at (42.4, 62.2)
- added H7: MountingHole_Pad, MountingHole:MountingHole_2.2mm_M2_Pad_Via, F.Cu at (-42.4, 62.2)
- added H8: MountingHole_Pad, MountingHole:MountingHole_2.2mm_M2_Pad_Via, F.Cu at (-62.2, 42.4)
- added H9: MountingHole_Pad, MountingHole:MountingHole_2.2mm_M2_Pad_Via, F.Cu at (-6.05, -50.7)
- added JP1: Jumper_3_Bridged12, Connector_PinHeader_1.27mm:PinHeader_1x03_P1.27mm_Vertical, F.Cu at (155.8, 43.7)
- added JP2: Jumper_3_Bridged12, Connector_PinHeader_1.27mm:PinHeader_1x03_P1.27mm_Vertical, F.Cu at (87.5, 71.2)
- added JP3: Jumper_3_Bridged12, Connector_PinHeader_1.27mm:PinHeader_1x03_P1.27mm_Vertical, F.Cu at (79.8, 73.2)
- added JP4: Jumper_3_Bridged23, Connector_PinHeader_1.27mm:PinHeader_1x03_P1.27mm_Vertical, F.Cu at (96.8, 71.2)
- added JP5: Jumper_3_Bridged12, Connector_PinHeader_1.27mm:PinHeader_1x03_P1.27mm_Vertical, F.Cu at (101.4, 71.2)
- added JP6: Jumper_3_Bridged12, Connector_PinHeader_1.27mm:PinHeader_1x03_P1.27mm_Vertical, F.Cu at (106.1, 71.2)
- added JP7: Jumper_3_Bridged12, Connector_PinHeader_1.27mm:PinHeader_1x03_P1.27mm_Vertical, F.Cu at (110.7, 71.2)
- added JP8: Jumper_3_Bridged23, Connector_PinHeader_1.27mm:PinHeader_1x03_P1.27mm_Vertical, F.Cu at (115.4, 71.2)
- added R19: 4.7k, PCM_Resistor_SMD_AKL:R_0805_2012Metric_Pad1.15x1.40mm_HandSolder, B.Cu at (90.0, -50.5)
- added R20: 220R, PCM_Resistor_SMD_AKL:R_0805_2012Metric_Pad1.15x1.40mm_HandSolder, B.Cu at (90.0, -56.5)
- added R21: 4.7k, PCM_Resistor_SMD_AKL:R_0805_2012Metric_Pad1.15x1.40mm_HandSolder, B.Cu at (97.5, -37.0)
- added R22: 220R, PCM_Resistor_SMD_AKL:R_0805_2012Metric_Pad1.15x1.40mm_HandSolder, B.Cu at (97.5, -43.0)
- added R23: 4.7k, PCM_Resistor_SMD_AKL:R_0805_2012Metric_Pad1.15x1.40mm_HandSolder, B.Cu at (102.5, -22.0)
- added R24: 220R, PCM_Resistor_SMD_AKL:R_0805_2012Metric_Pad1.15x1.40mm_HandSolder, B.Cu at (102.5, -28.0)
- added R25: 4.7k, PCM_Resistor_SMD_AKL:R_0805_2012Metric_Pad1.15x1.40mm_HandSolder, B.Cu at (105.5, -5.50)
- added R26: 220R, PCM_Resistor_SMD_AKL:R_0805_2012Metric_Pad1.15x1.40mm_HandSolder, B.Cu at (105.5, -11.5)
- added R27: 4.7k, PCM_Resistor_SMD_AKL:R_0805_2012Metric_Pad1.15x1.40mm_HandSolder, B.Cu at (105.5, 5.50)
- added R28: 220R, PCM_Resistor_SMD_AKL:R_0805_2012Metric_Pad1.15x1.40mm_HandSolder, B.Cu at (105.5, 11.5)
- added R29: 4.7k, PCM_Resistor_SMD_AKL:R_0805_2012Metric_Pad1.15x1.40mm_HandSolder, B.Cu at (102.5, 22.0)
- added R30: 220R, PCM_Resistor_SMD_AKL:R_0805_2012Metric_Pad1.15x1.40mm_HandSolder, B.Cu at (102.5, 28.0)
- added R31: 4.7k, PCM_Resistor_SMD_AKL:R_0805_2012Metric_Pad1.15x1.40mm_HandSolder, B.Cu at (97.5, 37.0)
- added R32: 220R, PCM_Resistor_SMD_AKL:R_0805_2012Metric_Pad1.15x1.40mm_HandSolder, B.Cu at (97.5, 43.0)
- added R33: 4.7k, PCM_Resistor_SMD_AKL:R_0805_2012Metric_Pad1.15x1.40mm_HandSolder, B.Cu at (90.0, 50.5)
- added R34: 220R, PCM_Resistor_SMD_AKL:R_0805_2012Metric_Pad1.15x1.40mm_HandSolder, B.Cu at (90.0, 56.5)
- added R83: 4.7k, PCM_Resistor_SMD_AKL:R_0805_2012Metric_Pad1.15x1.40mm_HandSolder, B.Cu at (-74.0, -51.0)
- added R84: 220R, PCM_Resistor_SMD_AKL:R_0805_2012Metric_Pad1.15x1.40mm_HandSolder, B.Cu at (-74.0, -57.0)
- added R85: 4.7k, PCM_Resistor_SMD_AKL:R_0805_2012Metric_Pad1.15x1.40mm_HandSolder, B.Cu at (-66.5, -58.5)
- added R86: 220R, PCM_Resistor_SMD_AKL:R_0805_2012Metric_Pad1.15x1.40mm_HandSolder, B.Cu at (-66.5, -64.5)
- added R87: 4.7k, PCM_Resistor_SMD_AKL:R_0805_2012Metric_Pad1.15x1.40mm_HandSolder, B.Cu at (-59.0, -66.0)
- added R88: 220R, PCM_Resistor_SMD_AKL:R_0805_2012Metric_Pad1.15x1.40mm_HandSolder, B.Cu at (-59.0, -72.0)
- added R89: 4.7k, PCM_Resistor_SMD_AKL:R_0805_2012Metric_Pad1.15x1.40mm_HandSolder, B.Cu at (-51.5, -73.5)
- added R90: 220R, PCM_Resistor_SMD_AKL:R_0805_2012Metric_Pad1.15x1.40mm_HandSolder, B.Cu at (-51.5, -79.5)
- added R91: 4.7k, PCM_Resistor_SMD_AKL:R_0805_2012Metric_Pad1.15x1.40mm_HandSolder, B.Cu at (-54.0, -91.5)
- added R92: 220R, PCM_Resistor_SMD_AKL:R_0805_2012Metric_Pad1.15x1.40mm_HandSolder, B.Cu at (-48.0, -91.5)
- added R93: 4.7k, PCM_Resistor_SMD_AKL:R_0805_2012Metric_Pad1.15x1.40mm_HandSolder, B.Cu at (-40.0, -80.0)
- added R94: 220R, PCM_Resistor_SMD_AKL:R_0805_2012Metric_Pad1.15x1.40mm_HandSolder, B.Cu at (-34.0, -80.0)
- added R95: 4.7k, PCM_Resistor_SMD_AKL:R_0805_2012Metric_Pad1.15x1.40mm_HandSolder, B.Cu at (-28.0, -71.0)
- added R96: 220R, PCM_Resistor_SMD_AKL:R_0805_2012Metric_Pad1.15x1.40mm_HandSolder, B.Cu at (-22.0, -71.0)
- added R97: 4.7k, PCM_Resistor_SMD_AKL:R_0805_2012Metric_Pad1.15x1.40mm_HandSolder, B.Cu at (-12.0, -65.0)
- added R98: 220R, PCM_Resistor_SMD_AKL:R_0805_2012Metric_Pad1.15x1.40mm_HandSolder, B.Cu at (-6.00, -65.0)
- added SW1: MT-0-102-A101-M200-RS+PJ, EasyEDA:SW-TH_MT-0-103-A101-M200-RS, F.Cu at (-16.5, 14.8)
- added SW2: TS4535TP 250GF 009, EasyEDA:SW-SMD_4P-L4.5-W4.5-P3.00-LS6.8, F.Cu at (-12.2, 91.2)
- added SW3: TS4535TP 250GF 009, EasyEDA:SW-SMD_4P-L4.5-W4.5-P3.00-LS6.8, F.Cu at (12.5, 91.2)
- AMUX1, AMUX2, AMUX3, C4, LDO1, MOUSE_FPC1, MOUSE_FPC2: moved to B.Cu
- C2: renamed from C3; moved to B.Cu
- C3: renamed from C2; moved to B.Cu
- R1: renamed from R13; value 4.7k -> 2.7K
- R2: renamed from R14; value 220R -> 2.7K
- R35: renamed from R51; value DNP -> 4.7k; moved to B.Cu
- R36: renamed from R52; value 0R -> 220R; moved to B.Cu
- R37: renamed from R53; value DNP -> 4.7k; moved to B.Cu
- R38: renamed from R54; value 0R -> 220R; moved to B.Cu
- R39: renamed from R55; value DNP -> 4.7k; moved to B.Cu
- R40: renamed from R56; value 0R -> 220R; moved to B.Cu
- R41: renamed from R57; value DNP -> 4.7k; moved to B.Cu
- R42: renamed from R58; value 0R -> 220R; moved to B.Cu
- R43: renamed from R59; value 2.7K -> 4.7k; moved to B.Cu
- R44: renamed from R60; value 2.7K -> 220R; moved to B.Cu
- R45: renamed from R61; value 0R -> 4.7k; moved to B.Cu
- R46: renamed from R62; value DNP -> 220R; moved to B.Cu
- R47: renamed from R63; value DNP -> 4.7k; moved to B.Cu
- R48: renamed from R64; value 0R -> 220R; moved to B.Cu
- R49: renamed from R65; value DNP -> 4.7k; moved to B.Cu
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- renumbered U1 to MCU1, R26 to R10, R27 to R11, R28 to R12, R29 to R13, R30 to R14, R31 to R15, R32 to R16, R33 to R17, R34 to R18, R19 to R3, R20 to R4, R21 to R5, R67 to R51, R68 to R52, R69 to R53, R70 to R54, R71 to R55, R72 to R56, R73 to R57, R74 to R58, R75 to R59, R22 to R6, R76 to R60, R77 to R61, R78 to R62, R79 to R63, R80 to R64, R81 to R65, R82 to R66, R83 to R67, R84 to R68, R85 to R69, R23 to R7, R86 to R70, R87 to R71, R88 to R72, R89 to R73, R90 to R74, R91 to R75, R92 to R76, R93 to R77, R94 to R78, R95 to R79, R24 to R8, R96 to R80, R97 to R81, R98 to R82, R25 to R9
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Connections:
- BUCK1 pad 1: VCC -> Net-(BUCK1-IN+)
- C1 pad 1: GND -> Net-(BUCK1-IN+)
- C1 pad 2: VCC -> GND
- C2 pad 2: unconnected-(C3-Pad2) -> +5V
- C3 pad 1: unconnected-(C2-Pad1) -> GND
- C4 pad 1: unconnected-(C4-Pad1) -> GND
- DRV1 pad 10: /DRV1_IPROPI -> /DRV5_IPROPI
- DRV1 pad 11: /DRV1_NSLEEP -> /DRV5_NSLEEP
- DRV1 pad 2: /DRV1_SCS -> /DRV5_SCS
- DRV1 pad 3: /DRV1_IN2 -> /DRV5_IN2
- DRV1 pad 4: /DRV1_IN1 -> /DRV5_IN1
- DRV1 pad 5: /DRV1_OFF -> /DRV5_OFF
- DRV1 pad 9: /DRV1_NFAULT -> /DRV5_NFAULT
- DRV2 pad 10: /DRV2_IPROPI -> /DRV4_IPROPI
- DRV2 pad 11: /DRV2_NSLEEP -> /DRV4_NSLEEP
- DRV2 pad 2: /DRV2_SCS -> /DRV4_SCS
- DRV2 pad 3: /DRV2_IN2 -> /DRV4_IN2
- DRV2 pad 4: /DRV2_IN1 -> /DRV4_IN1
- DRV2 pad 5: /DRV2_OFF -> /DRV4_OFF
- DRV2 pad 9: /DRV2_NFAULT -> /DRV4_NFAULT
- DRV4 pad 10: /DRV4_IPROPI -> /DRV2_IPROPI
- DRV4 pad 11: /DRV4_NSLEEP -> /DRV2_NSLEEP
- DRV4 pad 2: /DRV4_SCS -> /DRV2_SCS
- DRV4 pad 3: /DRV4_IN2 -> /DRV2_IN2
- DRV4 pad 4: /DRV4_IN1 -> /DRV2_IN1
- DRV4 pad 5: /DRV4_OFF -> /DRV2_OFF
- DRV4 pad 9: /DRV4_NFAULT -> /DRV2_NFAULT
- DRV5 pad 10: /DRV5_IPROPI -> /DRV1_IPROPI
- DRV5 pad 11: /DRV5_NSLEEP -> /DRV1_NSLEEP
- DRV5 pad 2: /DRV5_SCS -> /DRV1_SCS
- DRV5 pad 3: /DRV5_IN2 -> /DRV1_IN2
- DRV5 pad 4: /DRV5_IN1 -> /DRV1_IN1
- DRV5 pad 5: /DRV5_OFF -> /DRV1_OFF
- DRV5 pad 9: /DRV5_NFAULT -> /DRV1_NFAULT
- PR1 pad 2: /line sensor array 1/LS2 -> /line sensor array 1/LS1
- PR11 pad 2: /line sensor array 1/LS15 -> /line sensor array 1/LS11
- PR12 pad 2: /line sensor array 1/LS16 -> /line sensor array 1/LS12
- PR13 pad 2: /line sensor array 1/LS11 -> /line sensor array 1/LS13
- PR14 pad 2: /line sensor array 1/LS12 -> /line sensor array 1/LS14
- PR15 pad 2: /line sensor array 1/LS13 -> /line sensor array 1/LS15
- PR16 pad 2: /line sensor array 1/LS14 -> /line sensor array 1/LS16
- PR17 pad 2: /line sensor array 2/LS2 -> /line sensor array 2/LS1
- PR18 pad 2: /line sensor array 2/LS1 -> /line sensor array 2/LS2
- PR19 pad 2: /line sensor array 2/LS8 -> /line sensor array 2/LS3
- PR2 pad 2: /line sensor array 1/LS1 -> /line sensor array 1/LS2
- PR20 pad 2: /line sensor array 2/LS7 -> /line sensor array 2/LS4
- PR21 pad 2: /line sensor array 2/LS4 -> /line sensor array 2/LS5
- PR22 pad 2: /line sensor array 2/LS3 -> /line sensor array 2/LS6
- PR23 pad 2: /line sensor array 2/LS5 -> /line sensor array 2/LS7
- PR24 pad 2: /line sensor array 2/LS6 -> /line sensor array 2/LS8
- PR27 pad 2: /line sensor array 2/LS15 -> /line sensor array 2/LS11
- PR28 pad 2: /line sensor array 2/LS16 -> /line sensor array 2/LS12
- PR29 pad 2: /line sensor array 2/LS11 -> /line sensor array 2/LS13
- PR3 pad 2: /line sensor array 1/LS8 -> /line sensor array 1/LS3
- PR30 pad 2: /line sensor array 2/LS12 -> /line sensor array 2/LS14
- PR31 pad 2: /line sensor array 2/LS13 -> /line sensor array 2/LS15
- PR32 pad 2: /line sensor array 2/LS14 -> /line sensor array 2/LS16
- PR33 pad 2: /line sensor array 3/LS2 -> /line sensor array 3/LS1
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Routing:
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- added copper zone on F.Cu, net VCC
Other:
- outline, holes or cut-outs redrawn
