File: hardware/bottom-plate/pcb/pcb.kicad_sch (KiCad schematic)
At the start: 58 parts, among them SW1 MT-0-102-A101-M200-RS+PJ, SW2 TS4535TP 250GF 009, SW3 TS4535TP 250GF 009

Commit message: completed bottom pcb
Parts:
- H10, H9: footprint MountingHole:MountingHole_2.2mm_M2_Pad_Via -> MountingHole:MountingHole_3.2mm_M3_Pad_Via
- renumbered DMUX2 to DMUX1, DMUX1 to DMUX2, JP5 to JP2, JP6 to JP3, JP2 to JP5, JP3 to JP6
Connections:
- net ADC_INT1: now also DMUX2.2 (GPB1); no longer DMUX1.6 (GPB5)
- net ADC_INT2: now also DMUX2.3 (GPB2); no longer DMUX1.7 (GPB6)
- net AMUX1_COM: now also MCU1.34 (GPIO28_ADC2); no longer MCU1.31 (GPIO26_ADC0)
- net AMUX3_COM: now also MCU1.31 (GPIO26_ADC0); no longer MCU1.34 (GPIO28_ADC2)
- net AMUX_EN: now also DMUX1.26 (GPA5); no longer DMUX1.28 (GPA7)
- net AMUX_S0: now also DMUX1.28 (GPA7); no longer DMUX2.25 (GPA4)
- net AMUX_S1: now also DMUX1.27 (GPA6); no longer DMUX2.26 (GPA5)
- net AMUX_S2: now also DMUX1.25 (GPA4); no longer DMUX2.27 (GPA6)
- net AMUX_S3: now also DMUX1.24 (GPA3); no longer DMUX2.28 (GPA7)
- net DMUX1_INT: now also DMUX1.20 (INTA), DMUX2.6 (GPB5); no longer DMUX2.20 (INTA), MCU1.25 (GPIO19)
- net DMUX2_INT: now also DMUX2.20 (INTA), MCU1.14 (GPIO10); no longer DMUX1.20 (INTA), DMUX1.8 (GPB7)
- net DMUX_RESET: now also MCU1.19 (GPIO14); no longer MCU1.26 (GPIO20)
- net DMUX_SCS: now also MCU1.7 (GPIO5); no longer MCU1.27 (GPIO21)
- net DRV1_IN1: now also MCU1.24 (GPIO18); no longer MCU1.9 (GPIO6)
- net DRV1_IN2: now also MCU1.25 (GPIO19); no longer MCU1.10 (GPIO7)
- net DRV1_NFAULT: now also DMUX2.4 (GPB3); no longer DMUX1.1 (GPB0)
- net DRV1_NSLEEP: now also DMUX1.3 (GPB2); no longer DMUX2.2 (GPB1)
- net DRV1_OFF: now also DMUX1.1 (GPB0); no longer DMUX2.1 (GPB0)
- net DRV1_SCS: now also DMUX1.2 (GPB1); no longer DMUX1.21 (GPA0)
- net DRV2_IN1: now also MCU1.1 (GPIO0); no longer MCU1.11 (GPIO8)
- net DRV2_IN2: now also MCU1.2 (GPIO1); no longer MCU1.12 (GPIO9)
- net DRV2_NFAULT: now also DMUX2.21 (GPA0); no longer DMUX1.2 (GPB1)
- net DRV2_NSLEEP: now also DMUX2.22 (GPA1); no longer DMUX2.4 (GPB3)
- net DRV2_OFF: now also DMUX2.7 (GPB6); no longer DMUX2.3 (GPB2)
- net DRV2_SCS: now also DMUX2.8 (GPB7); no longer DMUX1.22 (GPA1)
- net DRV3_IN1: now also MCU1.11 (GPIO8); no longer MCU1.14 (GPIO10)
- net DRV3_IN2: now also MCU1.12 (GPIO9); no longer MCU1.15 (GPIO11)
- net DRV3_IPROPI: now also ADC1.6 (AIN2); no longer ADC1.7 (AIN3)
- net DRV3_NFAULT: now also DMUX2.28 (GPA7); no longer DMUX1.3 (GPB2)
- net DRV3_NSLEEP: now also DMUX2.27 (GPA6); no longer DMUX2.6 (GPB5)
- net DRV3_OFF: now also DMUX2.26 (GPA5); no longer DMUX2.5 (GPB4)
- net DRV3_SCS: now also DMUX2.25 (GPA4); no longer DMUX1.23 (GPA2)
- net DRV4_IN1: now also MCU1.26 (GPIO20); no longer MCU1.16 (GPIO12)
- net DRV4_IN2: now also MCU1.27 (GPIO21); no longer MCU1.17 (GPIO13)
- net DRV4_NFAULT: now also DMUX2.5 (GPB4); no longer DMUX1.4 (GPB3)
- net DRV4_NSLEEP: now also DMUX1.7 (GPB6); no longer DMUX2.8 (GPB7)
- net DRV4_OFF: now also DMUX1.21 (GPA0); no longer DMUX2.7 (GPB6)
- net DRV4_SCS: now also DMUX1.8 (GPB7); no longer DMUX1.24 (GPA3)
- net DRV5_IN1: now also MCU1.16 (GPIO12); no longer MCU1.19 (GPIO14)
- net DRV5_IN2: now also MCU1.17 (GPIO13); no longer MCU1.20 (GPIO15)
- net DRV5_IPROPI: now also ADC1.7 (AIN3); no longer ADC1.6 (AIN2)
- net DRV5_NFAULT: now also DMUX2.1 (GPB0); no longer DMUX1.5 (GPB4)
- net DRV5_NSLEEP: now also DMUX1.6 (GPB5); no longer DMUX1.27 (GPA6)
- net DRV5_OFF: now also DMUX1.5 (GPB4); no longer DMUX1.26 (GPA5)
- net DRV5_SCS: now also DMUX1.4 (GPB3); no longer DMUX1.25 (GPA4)
- net I2C0.SCL: now also MCU1.10 (GPIO7); no longer MCU1.2 (GPIO1)
- net I2C0.SDA: now also MCU1.9 (GPIO6); no longer MCU1.1 (GPIO0)
- net KICK: now also MCU1.20 (GPIO15); no longer MCU1.24 (GPIO18)
- net MOUSE1_RST: now also DMUX1.22 (GPA1); no longer DMUX2.23 (GPA2)
- net MOUSE1_SCS: now also DMUX1.23 (GPA2); no longer DMUX2.21 (GPA0)
- net MOUSE2_MOT: now also MCU1.15 (GPIO11); no longer MCU1.7 (GPIO5)
- net MOUSE2_RST: now also DMUX2.23 (GPA2); no longer DMUX2.24 (GPA3)
- net MOUSE2_SCS: now also DMUX2.24 (GPA3); no longer DMUX2.22 (GPA1)
- net at JP1.2 (C): now also DMUX1.15 (A0); no longer DMUX2.15 (A0)
- net at JP4.2 (C): now also DMUX2.15 (A0); no longer DMUX1.15 (A0)
Other:
- moved on the sheet: DMUX1, DMUX2, JP2, JP3, JP5, JP6

Commit message: added testpoints and fixed issues with bottom plate
Parts:
- added 3V3TP1, 5VTP1, GNDTP1, GNDTP2, VCCTP1: TestPoint, TestPoint:TestPoint_THTPad_D1.0mm_Drill0.5mm, symbol Connector:TestPoint
- added C5: 470uF, Capacitor_SMD:CP_Elec_6.3x7.7, symbol Device:C_Polarized
- added ESC1: Conn_01x03, Connector_JST:JST_XH_B3B-XH-A_1x03_P2.50mm_Vertical, symbol Connector_Generic:Conn_01x03
- added PWR3: XT30-F, Connector_AMASS:AMASS_XT30U-F_1x02_P5.0mm_Vertical, symbol Connector_Generic:Conn_01x02
- C1: value 150uF -> 100uF
Connections:
- net +3V3: now also 3V3TP1.1
- net +5V: now also 5VTP1.1
- net DRV5_IN1: now also ESC1.3 (Pin_3)
- net DRV5_IN2: now also ESC1.2 (Pin_2)
- net GND: now also C5.2, ESC1.1 (Pin_1), GNDTP1.1, GNDTP2.1, PWR3.1 (Pin_1)
- net VCC: now also C5.1, PWR3.2 (Pin_2), VCCTP1.1
Other:
- note added: "100uF to critically damp plug-in spike"
- note added: "Power to brushless motor ESC. DNP DRV5 if using brushless, and tape driver onto bottom plate."
- note added: "power"
- note removed: "150uF to critically damp plug-in spike"
