File: hardware/bottom-plate/pcb/line-sensor-array-1.kicad_sch (KiCad schematic)
At the start: 1 part

Commit message: completed bottom pcb
Parts:
- renumbered AMUX3 to AMUX1
Connections:
- net LS1: now also AMUX1.9 (I0); no longer AMUX1.2 (I7)
- net LS10: now also AMUX1.17 (I14); no longer AMUX1.22 (I9)
- net LS11: now also AMUX1.18 (I13); no longer AMUX1.21 (I10)
- net LS12: now also AMUX1.19 (I12); no longer AMUX1.20 (I11)
- net LS13: now also AMUX1.20 (I11); no longer AMUX1.19 (I12)
- net LS14: now also AMUX1.21 (I10); no longer AMUX1.18 (I13)
- net LS15: now also AMUX1.22 (I9); no longer AMUX1.17 (I14)
- net LS16: now also AMUX1.23 (I8); no longer AMUX1.16 (I15)
- net LS2: now also AMUX1.8 (I1); no longer AMUX1.3 (I6)
- net LS3: now also AMUX1.7 (I2); no longer AMUX1.4 (I5)
- net LS4: now also AMUX1.6 (I3); no longer AMUX1.5 (I4)
- net LS5: now also AMUX1.5 (I4); no longer AMUX1.6 (I3)
- net LS6: now also AMUX1.4 (I5); no longer AMUX1.7 (I2)
- net LS7: now also AMUX1.3 (I6); no longer AMUX1.8 (I1)
- net LS8: now also AMUX1.2 (I7); no longer AMUX1.9 (I0)
- net LS9: now also AMUX1.16 (I15); no longer AMUX1.23 (I8)
Changed lines of the file:
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@@
+		)
+	)
+	(label "LS13"
+		(at 95.25 100.33 180)
+		(fields_autoplaced yes)
+		(effects
+			(font
+				(size 1.27 1.27)
+			)
+			(justify right bottom)
 		)
 	)
@@
 		)
 	)
+	(label "LS2"
+		(at 95.25 74.93 180)
+		(fields_autoplaced yes)
+		(effects
+			(font
+				(size 1.27 1.27)
+			)
+			(justify right bottom)
+		)
+	)
 	(label "LS12"
 		(at 137.16 140.97 180)
@@
 		)
 	)
-	(label "LS1"
+	(label "LS8"
 		(at 95.25 90.17 180)
 		(fields_autoplaced yes)
@@
 		)
 	)
-	(label "LS13"
-		(at 95.25 102.87 180)
-		(fields_autoplaced yes)
-		(effects
-			(font
-				(size 1.27 1.27)
-			)
-			(justify right bottom)
-		)
-	)
-	(label "LS14"
-		(at 95.25 105.41 180)
-		(fields_autoplaced yes)
-		(effects
-			(font
-				(size 1.27 1.27)
-			)
-			(justify right bottom)
-		)
-	)
-	(label "LS6"
-		(at 95.25 77.47 180)
+	(label "LS4"
+		(at 95.25 80.01 180)
 		(fields_autoplaced yes)
 		(effects
@@
 		)
 	)
-	(label "LS4"
+	(label "LS5"
 		(at 95.25 82.55 180)
 		(fields_autoplaced yes)
@@
 		)
 	)
-	(label "LS11"
-		(at 95.25 97.79 180)
-		(fields_autoplaced yes)
-		(effects
-			(font
-				(size 1.27 1.27)
-			)
-			(justify right bottom)
-		)
-	)
-	(label "LS15"
+	(label "LS10"
 		(at 95.25 107.95 180)
 		(fields_autoplaced yes)
@@
 		)
 	)
-	(label "LS8"
-		(at 95.25 72.39 180)
-		(fields_autoplaced yes)
-		(effects
-			(font
-				(size 1.27 1.27)
-			)
-			(justify right bottom)
-		)
-	)
-	(label "LS10"
-		(at 95.25 95.25 180)
+	(label "LS7"
+		(at 95.25 87.63 180)
 		(fields_autoplaced yes)
 		(effects
@@
 		)
 	)
+	(label "LS3"
+		(at 95.25 77.47 180)
+		(fields_autoplaced yes)
+		(effects
+			(font
+				(size 1.27 1.27)
+			)
+			(justify right bottom)
+		)
+	)
 	(label "LS9"
 		(at 137.16 110.49 180)
@@
 		)
 	)
-	(label "LS2"
-		(at 95.25 87.63 180)
-		(fields_autoplaced yes)
-		(effects
-			(font
-				(size 1.27 1.27)
-			)
-			(justify right bottom)
-		)
-	)
 	(label "LS7"
 		(at 137.16 90.17 180)
@@
 		)
 	)
-	(label "LS16"
+	(label "LS9"
 		(at 95.25 110.49 180)
-		(fields_autoplaced yes)
-		(effects
-			(font
-				(size 1.27 1.27)
-			)
-			(justify right bottom)
-		)
-	)
-	(label "LS3"
-		(at 95.25 85.09 180)
 		(fields_autoplaced yes)
 		(effects
@@
 		)
 	)
-	(label "LS7"
-		(at 95.25 74.93 180)
+	(label "LS15"
+		(at 95.25 95.25 180)
 		(fields_autoplaced yes)
 		(effects
@@
 		)
 	)
+	(label "LS1"
+		(at 95.25 72.39 180)
+		(fields_autoplaced yes)
+		(effects
+			(font
+				(size 1.27 1.27)
+			)
+			(justify right bottom)
+		)
+	)
+	(label "LS14"
+		(at 95.25 97.79 180)
+		(fields_autoplaced yes)
+		(effects
+			(font
+				(size 1.27 1.27)
+			)
+			(justify right bottom)
+		)
+	)
 	(label "LS12"
-		(at 95.25 100.33 180)
-		(fields_autoplaced yes)
-		(effects
-			(font
-				(size 1.27 1.27)
-			)
-			(justify right bottom)
-		)
-	)
-	(label "LS5"
-		(at 95.25 80.01 180)
+		(at 95.25 102.87 180)
+		(fields_autoplaced yes)
+		(effects
+			(font
+				(size 1.27 1.27)
+			)
+			(justify right bottom)
+		)
+	)
+	(label "LS16"
+		(at 95.25 92.71 180)
+		(fields_autoplaced yes)
+		(effects
+			(font
+				(size 1.27 1.27)
+			)
+			(justify right bottom)
+		)
+	)
+	(label "LS11"
+		(at 95.25 105.41 180)
 		(fields_autoplaced yes)
 		(effects
@@
 		)
 	)
-	(label "LS9"
-		(at 95.25 92.71 180)
+	(label "LS6"
+		(at 95.25 85.09 180)
 		(fields_autoplaced yes)
 		(effects
@@
 		(dnp no)
 		(fields_autoplaced yes)
-		(property "Reference" "#PWR0211"
+		(property "Reference" "#PWR079"
 			(at 81.28 63.5 0)
 			(effects
@@
 		(instances
 			(project "pcb"
-				(path "/7e6d4b79-c480-4b70-bccc-d28260cddf7c/93e6d7bb-95f9-4cf2-95f4-5cf0dae1bc31"
-					(reference "#PWR0211")
-					(unit 1)
-				)
-				(path "/7e6d4b79-c480-4b70-bccc-d28260cddf7c/c980f11d-c85b-4c7f-a7ac-bfc985564f96"
-					(reference "#PWR0145")
-					(unit 1)
-				)
 				(path "/7e6d4b79-c480-4b70-bccc-d28260cddf7c/dd019f33-6d81-4ff9-8ccf-108909809042"
 					(reference "#PWR079")
@@
 		(dnp no)
 		(fields_autoplaced yes)
-		(property "Reference" "AMUX3"
+		(property "Reference" "AMUX1"
 			(at 81.242 63.5 0)
 			(effects
@@
 		(instances
 			(project "pcb"
-				(path "/7e6d4b79-c480-4b70-bccc-d28260cddf7c/93e6d7bb-95f9-4cf2-95f4-5cf0dae1bc31"
-					(reference "AMUX3")
-					(unit 1)
-				)
-				(path "/7e6d4b79-c480-4b70-bccc-d28260cddf7c/c980f11d-c85b-4c7f-a7ac-bfc985564f96"
-					(reference "AMUX2")
-					(unit 1)
-				)
 				(path "/7e6d4b79-c480-4b70-bccc-d28260cddf7c/dd019f33-6d81-4ff9-8ccf-108909809042"
 					(reference "AMUX1")
@@
 		(dnp no)
 		(fields_autoplaced yes)
-		(property "Reference" "#PWR0212"
+		(property "Reference" "#PWR080"
 			(at 71.12 119.38 0)
 			(effects
@@
 		(instances
 			(project "pcb"
-				(path "/7e6d4b79-c480-4b70-bccc-d28260cddf7c/93e6d7bb-95f9-4cf2-95f4-5cf0dae1bc31"
-					(reference "#PWR0212")
-					(unit 1)
-				)
-				(path "/7e6d4b79-c480-4b70-bccc-d28260cddf7c/c980f11d-c85b-4c7f-a7ac-bfc985564f96"
-					(reference "#PWR0146")
-					(unit 1)
-				)
 				(path "/7e6d4b79-c480-4b70-bccc-d28260cddf7c/dd019f33-6d81-4ff9-8ccf-108909809042"
 					(reference "#PWR080")
@@
 					(page "3")
 				)
-				(path "/7e6d4b79-c480-4b70-bccc-d28260cddf7c/93e6d7bb-95f9-4cf2-95f4-5cf0dae1bc31"
-					(page "37")
-				)
-				(path "/7e6d4b79-c480-4b70-bccc-d28260cddf7c/c980f11d-c85b-4c7f-a7ac-bfc985564f96"
-					(page "20")
-				)
 			)
 		)
@@
 					(page "8")
 				)
-				(path "/7e6d4b79-c480-4b70-bccc-d28260cddf7c/93e6d7bb-95f9-4cf2-95f4-5cf0dae1bc31"
-					(page "42")
-				)
-				(path "/7e6d4b79-c480-4b70-bccc-d28260cddf7c/c980f11d-c85b-4c7f-a7ac-bfc985564f96"
-					(page "25")
-				)
 			)
 		)
@@
 					(page "18")
 				)
-				(path "/7e6d4b79-c480-4b70-bccc-d28260cddf7c/93e6d7bb-95f9-4cf2-95f4-5cf0dae1bc31"
-					(page "52")
-				)
-				(path "/7e6d4b79-c480-4b70-bccc-d28260cddf7c/c980f11d-c85b-4c7f-a7ac-bfc985564f96"
-					(page "35")
-				)
 			)
 		)
@@
 					(page "12")
 				)
-				(path "/7e6d4b79-c480-4b70-bccc-d28260cddf7c/93e6d7bb-95f9-4cf2-95f4-5cf0dae1bc31"
-					(page "46")
-				)
-				(path "/7e6d4b79-c480-4b70-bccc-d28260cddf7c/c980f11d-c85b-4c7f-a7ac-bfc985564f96"
-					(page "29")
-				)
 			)
 		)
@@
 					(page "10")
 				)
-				(path "/7e6d4b79-c480-4b70-bccc-d28260cddf7c/93e6d7bb-95f9-4cf2-95f4-5cf0dae1bc31"
-					(page "44")
-				)
-				(path "/7e6d4b79-c480-4b70-bccc-d28260cddf7c/c980f11d-c85b-4c7f-a7ac-bfc985564f96"
-					(page "27")
-				)
 			)
 		)
@@
 					(page "17")
 				)
-				(path "/7e6d4b79-c480-4b70-bccc-d28260cddf7c/93e6d7bb-95f9-4cf2-95f4-5cf0dae1bc31"
-					(page "51")
-				)
-				(path "/7e6d4b79-c480-4b70-bccc-d28260cddf7c/c980f11d-c85b-4c7f-a7ac-bfc985564f96"
-					(page "34")
-				)
 			)
 		)
@@
 					(page "15")
 				)
-				(path "/7e6d4b79-c480-4b70-bccc-d28260cddf7c/93e6d7bb-95f9-4cf2-95f4-5cf0dae1bc31"
-					(page "49")
-				)
-				(path "/7e6d4b79-c480-4b70-bccc-d28260cddf7c/c980f11d-c85b-4c7f-a7ac-bfc985564f96"
-					(page "32")
-				)
 			)
 		)
@@
 					(page "9")
 				)
-				(path "/7e6d4b79-c480-4b70-bccc-d28260cddf7c/93e6d7bb-95f9-4cf2-95f4-5cf0dae1bc31"
-					(page "43")
-				)
-				(path "/7e6d4b79-c480-4b70-bccc-d28260cddf7c/c980f11d-c85b-4c7f-a7ac-bfc985564f96"
-					(page "26")
-				)
 			)
 		)
@@
 					(page "5")
 				)
-				(path "/7e6d4b79-c480-4b70-bccc-d28260cddf7c/93e6d7bb-95f9-4cf2-95f4-5cf0dae1bc31"
-					(page "39")
-				)
-				(path "/7e6d4b79-c480-4b70-bccc-d28260cddf7c/c980f11d-c85b-4c7f-a7ac-bfc985564f96"
-					(page "22")
-				)
 			)
 		)
@@
 					(page "7")
 				)
-				(path "/7e6d4b79-c480-4b70-bccc-d28260cddf7c/93e6d7bb-95f9-4cf2-95f4-5cf0dae1bc31"
-					(page "41")
-				)
-				(path "/7e6d4b79-c480-4b70-bccc-d28260cddf7c/c980f11d-c85b-4c7f-a7ac-bfc985564f96"
-					(page "24")
-				)
 			)
 		)
@@
 					(page "11")
 				)
-				(path "/7e6d4b79-c480-4b70-bccc-d28260cddf7c/93e6d7bb-95f9-4cf2-95f4-5cf0dae1bc31"
-					(page "45")
-				)
-				(path "/7e6d4b79-c480-4b70-bccc-d28260cddf7c/c980f11d-c85b-4c7f-a7ac-bfc985564f96"
-					(page "28")
-				)
 			)
 		)
@@
 					(page "13")
 				)
-				(path "/7e6d4b79-c480-4b70-bccc-d28260cddf7c/93e6d7bb-95f9-4cf2-95f4-5cf0dae1bc31"
-					(page "47")
-				)
-				(path "/7e6d4b79-c480-4b70-bccc-d28260cddf7c/c980f11d-c85b-4c7f-a7ac-bfc985564f96"
-					(page "30")
-				)
 			)
 		)
@@
 					(page "6")
 				)
-				(path "/7e6d4b79-c480-4b70-bccc-d28260cddf7c/93e6d7bb-95f9-4cf2-95f4-5cf0dae1bc31"
-					(page "40")
-				)
-				(path "/7e6d4b79-c480-4b70-bccc-d28260cddf7c/c980f11d-c85b-4c7f-a7ac-bfc985564f96"
-					(page "23")
-				)
 			)
 		)
@@
 					(page "16")
 				)
-				(path "/7e6d4b79-c480-4b70-bccc-d28260cddf7c/93e6d7bb-95f9-4cf2-95f4-5cf0dae1bc31"
-					(page "50")
-				)
-				(path "/7e6d4b79-c480-4b70-bccc-d28260cddf7c/c980f11d-c85b-4c7f-a7ac-bfc985564f96"
-					(page "33")
-				)
 			)
 		)
@@
 					(page "14")
 				)
-				(path "/7e6d4b79-c480-4b70-bccc-d28260cddf7c/93e6d7bb-95f9-4cf2-95f4-5cf0dae1bc31"
-					(page "48")
-				)
-				(path "/7e6d4b79-c480-4b70-bccc-d28260cddf7c/c980f11d-c85b-4c7f-a7ac-bfc985564f96"
-					(page "31")
-				)
 			)
 		)
@@
 					(page "4")
 				)
-				(path "/7e6d4b79-c480-4b70-bccc-d28260cddf7c/93e6d7bb-95f9-4cf2-95f4-5cf0dae1bc31"
-					(page "38")
-				)
-				(path "/7e6d4b79-c480-4b70-bccc-d28260cddf7c/c980f11d-c85b-4c7f-a7ac-bfc985564f96"
-					(page "21")
-				)
-			)
+			)
