File: hardware/bottom-plate/pcb/line-sensor-array-2.kicad_sch (KiCad schematic)
At the start: 1 part

Commit message: completed bottom pcb
Parts:
- renumbered AMUX3 to AMUX2
Connections:
- net LS1: now also AMUX2.23 (I8); no longer AMUX2.2 (I7)
- net LS10: now also AMUX2.7 (I2); no longer AMUX2.22 (I9)
- net LS11: now also AMUX2.8 (I1); no longer AMUX2.21 (I10)
- net LS12: now also AMUX2.9 (I0); no longer AMUX2.20 (I11)
- net LS2: now also AMUX2.22 (I9); no longer AMUX2.3 (I6)
- net LS3: now also AMUX2.21 (I10); no longer AMUX2.4 (I5)
- net LS4: now also AMUX2.20 (I11); no longer AMUX2.5 (I4)
- net LS5: now also AMUX2.2 (I7); no longer AMUX2.6 (I3)
- net LS6: now also AMUX2.3 (I6); no longer AMUX2.7 (I2)
- net LS7: now also AMUX2.4 (I5); no longer AMUX2.8 (I1)
- net LS8: now also AMUX2.5 (I4); no longer AMUX2.9 (I0)
- net LS9: now also AMUX2.6 (I3); no longer AMUX2.23 (I8)
