File: hardware/top-plate/top-plate/CH201.kicad_sch (KiCad schematic)
At the start: 24 parts

Commit message: :sparkles: Done with top plate?
Parts:
- added C5: 1uF, PCM_Capacitor_SMD_AKL:C_0805_2012Metric_Pad1.15x1.40mm_HandSolder, symbol Device:C
- added U1: SN74LVC2T45DCUR, Package_SO:VSSOP-8_2.3x2mm_P0.5mm, symbol Logic_LevelTranslator:SN74LVC2T45DCUR
Connections:
- net +1V8: now also C5.2, U1.1 (VCCA), U1.5 (DIR)
- net +3V3: now also U1.8 (VCCB)
- net GND: now also C5.1, U1.4 (GND)
Other:
- note added: "Level Shifter"
- note added: "Sheet Pins"
- note removed: "All left as shape "input" for now, Possibly requires changing ltr"
- note removed: "Other Outputs"
- moved on the sheet: DMUX_INT, DMUX_PROG, FFC_US1, FFC_US10, FFC_US11, FFC_US12, FFC_US13, FFC_US14, FFC_US15, FFC_US16, FFC_US2, FFC_US3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
