File: hardware/top-plate/top-plate/top-plate.kicad_sch (KiCad schematic)
At the start: 19 parts

Commit message: :sparkles: Done with top plate?
Parts:
- added BUCK1: ~, custom:mini560, symbol custom:mini360/560
- added C1: 1uF, PCM_Capacitor_SMD_AKL:C_0805_2012Metric_Pad1.15x1.40mm_HandSolder, symbol Device:C
- added C2: 10uF, PCM_Capacitor_SMD_AKL:C_0805_2012Metric_Pad1.15x1.40mm_HandSolder, symbol Device:C
- added C3: 100uF, Capacitor_SMD:CP_Elec_6.3x7.7, symbol Device:C_Polarized
- added C4: 22uF, PCM_Capacitor_SMD_AKL:C_0805_2012Metric_Pad1.15x1.40mm_HandSolder, symbol Device:C
- added LDO1: TLV1117-33, Package_TO_SOT_SMD:SOT-223-3_TabPin2, symbol Regulator_Linear:TLV1117-33
- added LED1, LED10, LED13, LED14, LED15, LED16, LED19, LED2, LED20, LED21, LED22, LED3, LED4, LED7, LED8, LED9: WS2812B, LED_SMD:LED_WS2812B-Mini_PLCC4_3.5x3.5mm, symbol LED:WS2812B
- added PWR1: XT30-M, Connector_AMASS:AMASS_XT30U-M_1x02_P5.0mm_Vertical, symbol Connector_Generic:Conn_01x02
- added SW1: MT-0-102-A101-M200-RS+PJ, EasyEDA:SW-TH_MT-0-103-A101-M200-RS, symbol EasyEDA:MT-0-102-A101-M200-RS+PJ
Connections:
- net +3V3: now also C2.2, LDO1.2 (VO)
- net +5V: now also BUCK1.3 (OUT+), C1.2, C4.2, LDO1.3 (VI), LED1.1 (VDD), LED10.1 (VDD), LED13.1 (VDD), LED14.1 (VDD), LED15.1 (VDD), LED16.1 (VDD), LED19.1 (VDD), LED2.1 (VDD), LED20.1 (VDD), LED21.1 (VDD), LED22.1 (VDD), LED3.1 (VDD), LED4.1 (VDD), LED7.1 (VDD), LED8.1 (VDD), LED9.1 (VDD)
- net GND: now also BUCK1.2 (IN-), BUCK1.4 (OUT-), C1.1, C2.1, C3.2, C4.1, LDO1.1 (GND), LED1.3 (VSS), LED10.3 (VSS), LED13.3 (VSS), LED14.3 (VSS), LED15.3 (VSS), LED16.3 (VSS), LED19.3 (VSS), LED2.3 (VSS), LED20.3 (VSS), LED21.3 (VSS), LED22.3 (VSS), LED3.3 (VSS), LED4.3 (VSS), LED7.3 (VSS), LED8.3 (VSS), LED9.3 (VSS), PWR1.1 (Pin_1), SW1.3
- net INTA_INT: no longer MCU1.12 (GPIO9)
- net INTB_INT: now also MCU1.12 (GPIO9)
- net US_RST: now also MCU1.16 (GPIO12); no longer MCU1.29 (GPIO22)
- net LED_SIG_5V: now reaches MCU1.17 (GPIO13)
- net LED_SIG_5V: now also LED1.4 (DIN)
- new net: LED1.2 (DOUT), LED7.4 (DIN)
- new net: LED19.2 (DOUT), LED20.4 (DIN)
- new net: LED13.2 (DOUT), LED19.4 (DIN)
- new net: BUCK1.1 (IN+), C3.1, SW1.2
- new net: LED13.4 (DIN), LED7.2 (DOUT)
- new net: LED21.2 (DOUT), LED22.4 (DIN)
- new net: LED15.2 (DOUT), LED21.4 (DIN)
- new net: LED10.2 (DOUT), LED4.4 (DIN)
- new net: LED10.4 (DIN), LED16.2 (DOUT)
- new net: LED14.2 (DOUT), LED8.4 (DIN)
- new net: LED14.4 (DIN), LED20.2 (DOUT)
- new net: LED15.4 (DIN), LED9.2 (DOUT)
- new net: LED16.4 (DIN), LED22.2 (DOUT)
- new net: LED2.4 (DIN), LED8.2 (DOUT)
- new net: LED3.2 (DOUT), LED9.4 (DIN)
- new net: LED2.2 (DOUT), LED3.4 (DIN)
- new net VCC: PWR1.2 (Pin_2), SW1.1
- no-connect marks 23 -> 24
Other:
- note added: "100uF to critically damp plug-in spike"
- note added: "Cuz its cool ~LJY Providing visual feedback, same as the middle plate"
- note added: "Cuz its very cool ~Probably LJY Providing visual feedback, same as LEDs"
- note added: "Fancy LEDs"
- note added: "LCD"
- note added: "Level Shifter for 5V to 3V3"
- note added: "MINI560 reg, to have a (mostly) guarenteed-to-work and replacable-if-fried design. 5A is way overkill, but the 3A ones are quite sketchy."
- note added: "PWR_FLAGs"
- note added: "Power"
- note added: "Power from middle plate."
- moved on the sheet: H1, H10, H11, H12, H13, H14, H15, H16, H17, H18, H2, H3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
