File: hardware/middle-plate/pcb/pcb.kicad_pcb (KiCad board)
At the start: 2 copper layers, 218 x 205.7 mm, 113 parts, among them SW1 MT-0-102-A101-M200-RS+PJ, SW2 TS4535TP 250GF 009, SW3 TS4535TP 250GF 009, SW4 TS4535TP 250GF 009, SW5 TS4535TP 250GF 009, SW6 TS4535TP 250GF 009, SW7 TS4535TP 250GF 009

Commit message: boom explosion
Parts:
- added H17: MountingHole_Pad, MountingHole:MountingHole_2.2mm_M2_Pad_Via, F.Cu at (-5.50, -30.0)
- added H18: MountingHole_Pad, MountingHole:MountingHole_2.2mm_M2_Pad_Via, F.Cu at (5.00, -30.0)
- added H19: MountingHole_Pad, MountingHole:MountingHole_2.2mm_M2_Pad_Via, F.Cu at (0.00, -15.0)
- added H20: MountingHole_Pad, MountingHole:MountingHole_2.2mm_M2_Pad_Via, F.Cu at (41.0, 14.5)
- added H21: MountingHole_Pad, MountingHole:MountingHole_2.2mm_M2_Pad_Via, F.Cu at (-41.0, 14.5)
Routing:
- net /IR1: track 32.3 -> 35.1 mm
- net /LED_SIG_5V: track 49.6 -> 47.0 mm
- net /IR11: track 64.0 -> 65.1 mm

Commit message: fixed middle plate and added stuff to gitignore
Parts:
- moved H17 0.50 mm to (-5.00, -30.0)
Connections:
- H17 pad 1: (no net) -> unconnected-(H17-Pad1)_5
- H18 pad 1: (no net) -> unconnected-(H18-Pad1)_3
- H19 pad 1: (no net) -> unconnected-(H19-Pad1)_4
- H20 pad 1: (no net) -> unconnected-(H20-Pad1)_8
- H21 pad 1: (no net) -> unconnected-(H21-Pad1)
Routing:
- net /IR1: track 35.1 -> 33.8 mm
