File: hardware/ultrasound/pcb/pcb.kicad_pcb (KiCad board)
At the start: 2 copper layers, 14 x 14 mm, 5 parts

Commit message: fixed motor driver footprint (one header had markings on bottom surface for some reason), generated production files
Other:
- board text added: "CH201 module V0.1"
- board text added: "Team BotByWire"
Changed lines of the file:
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@@
 		(layer "Edge.Cuts")
+	)
+	(gr_text "Team BotByWire"
+		(at 6 8.6 0)
+		(layer "B.SilkS")
+		(effects
+			(font
+				(size 1 1)
+				(thickness 0.15)
+			)
+			(justify left bottom mirror)
+		)
+	)
+	(gr_text "CH201\nmodule\nV0.1"
+		(at 0 1.8 0)
+		(layer "B.SilkS")
+		(effects
+			(font
+				(size 1 1)
+				(thickness 0.15)
+			)
+			(justify bottom mirror)
+		)
 	)
 	(segment
