File: hardware/top-plate/pcb/pcb.kicad_pcb (KiCad board)
At the start: 2 copper layers, 130 x 130 mm, 104 parts, among them J1 Conn_01x02, SW1 SS-12D10L5, SW2 TS4535TP 250GF 009, SW3 TS4535TP 250GF 009

Commit message: changed tlv1117-33 to tlv1117-18 on top pcb for 1.8V LDO
Parts:
- LDO2: value TLV1117-33 -> TLV1117-18
